File: hardware/main/main.kicad_sch (KiCad schematic)
At the start: 110 parts, among them IC1 ICM-42688-P, IC10 PE64906B-Z, IC2 PAM2306DYPAA, IC3 CC1121RHBR, IC4 CC1190RGVR, IC5 TXE8116DGSR, IC6 PE64906B-Z, IC7 PE64906B-Z, IC8 PE64906B-Z, IC9 PE64906B-Z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

Commit message: pcb work
Parts:
- C1, C2, C22, C23, C3, C33, C34, C37, C38, C39, C40: footprint (none) -> Capacitor_SMD:C_0805_2012Metric
- C12, C13, C14, C15, C18, C19, C20, C21, C30, C31, C32, C35, C36, C6, C9: footprint (none) -> Capacitor_SMD:C_0201_0603Metric
Connections:
- net +3V3: no longer C34.2
- net GND: no longer C34.1
- net at C14.1: now also IC3.18 (TRX_SW), L7.2; no longer IC4.10 (LNA_OUT)
- new net: C14.2, IC4.10 (LNA_OUT)

Commit message: pcb work
Parts:
- removed L2: 3.3uH, symbol Device:L_Small
- added J6: Conn_01x01, Connector_Wire:SolderWire-0.5sqmm_1x01_D0.9mm_OD2.3mm, symbol Connector_Generic:Conn_01x01
- added L14: 3.3uH, Inductor_SMD:L_1210_3225Metric_Pad1.42x2.65mm_HandSolder, symbol Device:L_Small
- C10, C16, C28: footprint (none) -> Capacitor_SMD:C_0201_0603Metric
- C11, C24, C25, C4, C5: footprint (none) -> Capacitor_SMD:C_0402_1005Metric
- C26, C27: value 100nF -> 0.1uF; footprint (none) -> Capacitor_SMD:C_0201_0603Metric
- C7, C8: footprint (none) -> Capacitor_SMD:C_0805_2012Metric
- L1: footprint (none) -> Inductor_SMD:L_Changjiang_FTC201612S
- L3: footprint (none) -> Inductor_SMD:L_1210_3225Metric_Pad1.42x2.65mm_HandSolder
Connections:
- net +3V3: now also C1.2, C7.1, U1.59 (ADC_AVDD), L14.1; no longer C7.2
- net GND: now also C28.1, C5.1, C7.2; no longer C28.2, C5.2, C7.1
- net at IC3.6 (DCPL): now also C28.2; no longer C28.1
- net at U1.31 (XOUT), Y1.1: now also C5.2; no longer C5.1
- net at R3.1, U1.61 (VREG_AVDD): no longer C1.2, U1.59 (ADC_AVDD)
- net at IC2.8 (LX1): now also L14.2
- net at U3.1 (RF_IN): now also J6.1 (Pin_1)

Commit message: pcb work
Parts:
- removed L13: 2.2nH*, symbol Device:L_Small
- removed R24: 4.55k, symbol Device:R_Small
- added L2: 2.2nH*, Inductor_SMD:L_0402_1005Metric, symbol Device:L_Small
- L1: footprint Inductor_SMD:L_Changjiang_FTC201612S -> CC1121RHBR:L_0806_2016Metric
- L10, L11: footprint (none) -> Inductor_SMD:L_0201_0603Metric
- L12, L6, L7, L9: footprint (none) -> Inductor_SMD:L_0402_1005Metric
- L4, L5: footprint (none) -> Inductor_SMD:L_01005_0402Metric
- L8: footprint (none) -> Inductor_SMD:L_0805_2012Metric
- R16, R3: footprint (none) -> Resistor_SMD:R_1206_3216Metric
- R19: value R_Small -> 56k
- R25: value 4.55k -> 9.1k; footprint (none) -> Resistor_SMD:R_0201_0603Metric
Connections:
- net +BATT: now also R25.2
- net at J1.2 (Pin_2): now also R2.2; no longer R1.1
- net at J1.3 (Pin_3): now also R1.1; no longer R2.1
- net at U1.67 (USB_DP): now also R1.2; no longer R2.2
- net at IC8.8 (RF+_1), IC8.9 (RF+_2), L12.2: now also L2.1
- net at AE1.1 (A), IC6.8 (RF+_1), IC6.9 (RF+_2): now also L2.2
- net at U1.66 (USB_DM): now also R2.1; no longer R1.2

Commit message: pcb work
Parts:
- removed C17: 100pF, symbol Device:C_Small
- removed J11: Conn_01x08_Pin, symbol Connector:Conn_01x08_Pin
- added C41: 100pF, Capacitor_SMD:C_0201_0603Metric, symbol Device:C_Small
- added R24: 9.1k, Resistor_SMD:R_0201_0603Metric, symbol Device:R_Small
- added U4: LPS22DF, Package_LGA:ST_HLGA-10_2x2mm_P0.5mm_LayoutBorder3x2y, symbol Sensor_Pressure:LPS22DF
- D1, D2: footprint (none) -> LED_SMD:LED_0201_0603Metric
- J10, J5, J7, J8, J9: footprint (none) -> Connector_PinHeader_1.27mm:PinHeader_1x08_P1.27mm_Vertical
- J2: footprint Connector_PinHeader_2.54mm:PinHeader_2x04_P2.54mm_Vertical -> Connector_PinHeader_1.27mm:PinHeader_2x04_P1.27mm_Vertical
- J3: footprint (none) -> Connector_PinHeader_2.54mm:PinHeader_1x03_P2.54mm_Vertical
- R1, R15, R19, R2: footprint (none) -> Resistor_SMD:R_0402_1005Metric
- R27: footprint (none) -> Resistor_SMD:R_0201_0603Metric
- R7: value 4.55k -> 1k
- Y2: footprint (none) -> Crystal:Crystal_SMD_3225-4Pin_3.2x2.5mm
Connections:
- net +3V3: now also C41.2, R24.1, U4.1 (Vdd_IO), U4.10 (VDD); no longer R7.1
- net GND: now also R7.1, U4.3 (GND), U4.7 (INT_DRDY), U4.8 (GND_IO), U4.9 (GND); no longer R6.1
- net MISO: now also U4.5 (SA0)
- net MOSI: now also U4.4 (SDA)
- net SCLK: now also U4.2 (SCL); no longer IC3.19 (LNA_P), IC9.8 (RF+_1), IC9.9 (RF+_2), L4.2, L6.1
- net at C6.2, IC2.4 (FB1), R6.2: now also R24.2; no longer R7.2
- net at U1.36 (GPIO28): now also U4.6 (~{CS})
- net at L9.2, R14.1: now also C41.1
- new net: R6.1, R7.2
- new net: IC3.19 (LNA_P), IC9.8 (RF+_1), IC9.9 (RF+_2), L4.2, L6.1

Commit message: pcb work
Parts:
- R4: footprint (none) -> Resistor_SMD:R_0201_0603Metric
Changed lines of the file:
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@@
 			)
 		)
-		(property "Footprint" ""
+		(property "Footprint" "Resistor_SMD:R_0201_0603Metric"
 			(at 96.52 143.51 0)
 			(effects
