File: hardware/main/main.kicad_sch (KiCad schematic)
At the start: 111 parts, among them IC1 ICM-42688-P, IC10 PE64906B-Z, IC2 PAM2306DYPAA, IC3 CC1121RHBR, IC4 CC1190RGVR, IC5 TXE8116DGSR, IC6 PE64906B-Z, IC7 PE64906B-Z, IC8 PE64906B-Z, IC9 PE64906B-Z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

Commit message: ethan commit
Parts:
- R10, R11, R12, R13, R14, R17, R18, R20, R21, R22, R26, R4, R5, R6, R7, R8, R9: footprint (none) -> Resistor_SMD:R_0201_0603Metric
Changed lines of the file:
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@@
 			)
 		)
-		(property "Footprint" ""
+		(property "Footprint" "Resistor_SMD:R_0201_0603Metric"
 			(at 173.99 132.08 0)
 			(effects
@@
 			)
 		)
-		(property "Footprint" ""
+		(property "Footprint" "Resistor_SMD:R_0201_0603Metric"
 			(at 237.49 123.19 0)
 			(effects
@@
 			)
 		)
-		(property "Footprint" ""
+		(property "Footprint" "Resistor_SMD:R_0201_0603Metric"
 			(at 100.33 124.46 0)
 			(effects
@@
 			)
 		)
-		(property "Footprint" ""
+		(property "Footprint" "Resistor_SMD:R_0201_0603Metric"
 			(at 359.41 81.28 0)
 			(effects
@@
 			)
 		)
-		(property "Footprint" ""
+		(property "Footprint" "Resistor_SMD:R_0201_0603Metric"
 			(at 97.79 261.62 0)
 			(effects
@@
 			)
 		)
-		(property "Footprint" ""
+		(property "Footprint" "Resistor_SMD:R_0201_0603Metric"
 			(at 180.34 129.54 0)
 			(effects
@@
 			)
 		)
-		(property "Footprint" ""
+		(property "Footprint" "Resistor_SMD:R_0201_0603Metric"
 			(at 90.17 248.92 0)
 			(effects
@@
 			)
 		)
-		(property "Footprint" ""
+		(property "Footprint" "Resistor_SMD:R_0201_0603Metric"
 			(at 240.03 133.35 0)
 			(effects
@@
 			)
 		)
-		(property "Footprint" ""
+		(property "Footprint" "Resistor_SMD:R_0201_0603Metric"
 			(at 240.03 128.27 0)
 			(effects
@@
 			)
 		)
-		(property "Footprint" ""
+		(property "Footprint" "Resistor_SMD:R_0201_0603Metric"
 			(at 213.36 66.04 0)
 			(effects
@@
 			)
 		)
-		(property "Footprint" ""
+		(property "Footprint" "Resistor_SMD:R_0201_0603Metric"
 			(at 363.22 83.82 0)
 			(effects
@@
 			)
 		)
-		(property "Footprint" ""
+		(property "Footprint" "Resistor_SMD:R_0201_0603Metric"
 			(at 367.03 78.74 0)
 			(effects
@@
 			)
 		)
-		(property "Footprint" ""
+		(property "Footprint" "Resistor_SMD:R_0201_0603Metric"
 			(at 377.19 124.46 0)
 			(effects
@@
 			)
 		)
-		(property "Footprint" ""
+		(property "Footprint" "Resistor_SMD:R_0201_0603Metric"
 			(at 100.33 250.19 0)
 			(effects
@@
 			)
 		)
-		(property "Footprint" ""
+		(property "Footprint" "Resistor_SMD:R_0201_0603Metric"
 			(at 96.52 143.51 0)
 			(effects
@@
 			)
 		)
-		(property "Footprint" ""
+		(property "Footprint" "Resistor_SMD:R_0201_0603Metric"
 			(at 200.66 64.77 0)
 			(effects
@@
 			)
 		)
-		(property "Footprint" ""
+		(property "Footprint" "Resistor_SMD:R_0201_0603Metric"
 			(at 102.87 246.38 0)
 			(effects

Commit message: pcb work
Parts:
- added C17, C42: 4.7uF, Capacitor_SMD:C_0805_2012Metric, symbol Device:C_Small
Connections:
- net +1V1: now also C17.2
- net +3V3: now also C34.2
- net GND: now also C34.1, U2.6 (GND), U2.7 (GND), C17.1, C42.1; no longer U2.6,7 (GND)
- net at R3.1, U1.61 (VREG_AVDD): now also C42.2
Other:
- moved on the sheet: C34

Commit message: pcb fixes
Connections:
- net +3V3: now also J10.3 (Pin_3), U1.38 (GPIO30), U1.68 (USB_OTP_VDD)
- net +5V: no longer U1.68 (USB_OTP_VDD)
- net GND: now also IC1.1 (AP_SDO_/_AP_AD0)
- net MOSI: now also C28.2, IC3.6 (DCPL), IC3.7 (SI), IC5.23 (SDI); no longer IC3.8 (SCLK), IC5.22 (SCLK)
- net SCLK: now also IC3.8 (SCLK), IC5.22 (SCLK); no longer IC3.7 (SI), IC5.23 (SDI)
Other:
- note added: "Codex hardware-fix labels"
