File: hardware/main/main.kicad_pcb (KiCad board)
At the start: 4 copper layers, 21 parts, among them IC1 ICM-42688-P, IC10 PE64906B-Z, IC2 PAM2306DYPAA, IC3 CC1121RHBR, IC4 CC1190RGVR, IC5 TXE8116DGSR, IC6 PE64906B-Z, IC7 PE64906B-Z, IC8 PE64906B-Z, IC9 PE64906B-Z, J1 USB-C, J2 Conn_01x08_Pin, J4 Conn_01x09, SW1 SW_Push, SW2 SW_Push, U1 RP2354B, U2 LSM6DSO32, U3 LG77LICMD, Y1 12MHz

Commit message: pcb work
Parts:
- added C1: 4.7uF, Capacitor_SMD:C_0805_2012Metric, F.Cu at (21.2, 58.5)
- added C10: 0.1uF, Capacitor_SMD:C_0201_0603Metric, F.Cu at (23.1, 25.0)
- added C11: 220pF, Capacitor_SMD:C_0402_1005Metric, F.Cu at (24.7, 25.3)
- added C12: 100pF, Capacitor_SMD:C_0201_0603Metric, F.Cu at (46.2, 67.5)
- added C13: 100pF, Capacitor_SMD:C_0201_0603Metric, F.Cu at (46.2, 69.2)
- added C14: 100pF, Capacitor_SMD:C_0201_0603Metric, F.Cu at (30.8, 29.4)
- added C15: 100pF, Capacitor_SMD:C_0201_0603Metric, F.Cu at (29.3, 30.4)
- added C16: 2.56pF, Capacitor_SMD:C_0201_0603Metric, F.Cu at (31.9, 31.8)
- added C18: 100pF, Capacitor_SMD:C_0201_0603Metric, F.Cu at (29.0, 19.7)
- added C19: 100pF, Capacitor_SMD:C_0201_0603Metric, F.Cu at (33.0, 20.1)
- added C2: 4.7uF, Capacitor_SMD:C_0805_2012Metric, F.Cu at (21.2, 61.5)
- added C20: 100pF, Capacitor_SMD:C_0201_0603Metric, F.Cu at (32.0, 19.0)
- added C21: 100pF, Capacitor_SMD:C_0201_0603Metric, F.Cu at (68.3, 83.7)
- added C22: 4.7uF, Capacitor_SMD:C_0805_2012Metric, F.Cu at (25.6, 58.5)
- added C23: 4.7uF, Capacitor_SMD:C_0805_2012Metric, F.Cu at (25.6, 61.5)
- added C24: 8pF, Capacitor_SMD:C_0402_1005Metric, F.Cu at (22.7, 20.9)
- added C25: 8pF, Capacitor_SMD:C_0402_1005Metric, F.Cu at (16.8, 22.2)
- added C26: 0.1uF, Capacitor_SMD:C_0201_0603Metric, F.Cu at (20.2, 24.7)
- added C27: 0.1uF, Capacitor_SMD:C_0201_0603Metric, F.Cu at (21.9, 24.4)
- added C28: 0.1uF, Capacitor_SMD:C_0201_0603Metric, F.Cu at (16.5, 29.3)
- added C3: 4.7uF, Capacitor_SMD:C_0805_2012Metric, F.Cu at (21.2, 64.5)
- added C30: 100pF, Capacitor_SMD:C_0201_0603Metric, F.Cu at (70.8, 78.5)
- added C31: 100pF, Capacitor_SMD:C_0201_0603Metric, F.Cu at (70.8, 80.2)
- added C32: 100pF, Capacitor_SMD:C_0201_0603Metric, F.Cu at (70.8, 82.0)
- added C33: 4.7uF, Capacitor_SMD:C_0805_2012Metric, F.Cu at (25.6, 64.5)
- added C34: 4.7uF, Capacitor_SMD:C_0805_2012Metric, F.Cu at (25.6, 67.5)
- added C35: 100pF, Capacitor_SMD:C_0201_0603Metric, F.Cu at (70.8, 83.7)
- added C36: 100pF, Capacitor_SMD:C_0201_0603Metric, F.Cu at (70.8, 85.5)
- added C37: 4.7uF, Capacitor_SMD:C_0805_2012Metric, F.Cu at (25.6, 70.5)
- added C38: 4.7uF, Capacitor_SMD:C_0805_2012Metric, F.Cu at (30.1, 58.5)
- added C39: 4.7uF, Capacitor_SMD:C_0805_2012Metric, F.Cu at (30.1, 61.5)
- added C4: 18pF, Capacitor_SMD:C_0402_1005Metric, F.Cu at (42.9, 16.9)
- added C40: 4.7uF, Capacitor_SMD:C_0805_2012Metric, F.Cu at (30.1, 64.5)
- added C41: 100pF, Capacitor_SMD:C_0201_0603Metric, F.Cu at (70.8, 87.2)
- added C5: 18pF, Capacitor_SMD:C_0402_1005Metric, F.Cu at (44.9, 16.9)
- added C6: 100pF, Capacitor_SMD:C_0201_0603Metric, F.Cu at (46.2, 62.2)
- added C7: 10uF, Capacitor_SMD:C_0805_2012Metric, F.Cu at (21.2, 67.5)
- added C8: 10uF, Capacitor_SMD:C_0805_2012Metric, F.Cu at (21.2, 70.5)
- added C9: 100pF, Capacitor_SMD:C_0201_0603Metric, F.Cu at (46.2, 64.0)
- added D1: White, LED_SMD:LED_0201_0603Metric, F.Cu at (79.7, 85.1)
- added D2: Blue, LED_SMD:LED_0201_0603Metric, F.Cu at (79.7, 86.9)
- added J10: Conn_01x08_Pin, Connector_PinHeader_1.27mm:PinHeader_1x08_P1.27mm_Vertical, F.Cu at (48.6, 1.77)
- added J3: Conn_01x03_Pin, Connector_PinHeader_2.54mm:PinHeader_1x03_P2.54mm_Vertical, F.Cu at (16.7, 84.2)
- added J5: Conn_01x08_Pin, Connector_PinHeader_1.27mm:PinHeader_1x08_P1.27mm_Vertical, F.Cu at (23.6, 1.85)
- added J6: Conn_01x01, Connector_Wire:SolderWire-0.5sqmm_1x01_D0.9mm_OD2.3mm, F.Cu at (1.65, 30.2)
- added J7: Conn_01x08_Pin, Connector_PinHeader_1.27mm:PinHeader_1x08_P1.27mm_Vertical, F.Cu at (60.1, 1.75)
- added J8: Conn_01x08_Pin, Connector_PinHeader_1.27mm:PinHeader_1x08_P1.27mm_Vertical, F.Cu at (60.2, 44.7)
- added J9: Conn_01x08_Pin, Connector_PinHeader_1.27mm:PinHeader_1x08_P1.27mm_Vertical, F.Cu at (36.6, 1.77)
- added L1: 3.3uH, CC1121RHBR:L_0806_2016Metric, F.Cu at (79.0, 102.4)
- added L10: 3.3nH*, Inductor_SMD:L_0201_0603Metric, F.Cu at (29.0, 18.3)
- added L11: 27nH, Inductor_SMD:L_0201_0603Metric, F.Cu at (73.2, 78.5)
- added L12: 2.2nH*, Inductor_SMD:L_0402_1005Metric, F.Cu at (22.8, 19.0)
- added L14: 3.3uH, Inductor_SMD:L_1210_3225Metric_Pad1.42x2.65mm_HandSolder, F.Cu at (77.4, 82.2)
- added L2: 2.2nH*, Inductor_SMD:L_0402_1005Metric, F.Cu at (17.1, 19.0)
- added L3: 3.3uH, Inductor_SMD:L_1210_3225Metric_Pad1.42x2.65mm_HandSolder, F.Cu at (77.4, 77.9)
- added L4: 18nH*, Inductor_SMD:L_01005_0402Metric, F.Cu at (24.9, 29.0)
- added L5: 18nH, Inductor_SMD:L_01005_0402Metric, F.Cu at (24.9, 27.8)
- added L6: 9.1nH*, Inductor_SMD:L_0402_1005Metric, F.Cu at (26.3, 29.3)
- added L7: 5.6nH, Inductor_SMD:L_0402_1005Metric, F.Cu at (28.2, 29.3)
- added L8: 10nH, Inductor_SMD:L_0805_2012Metric, F.Cu at (31.9, 30.6)
- added L9: 33nH, Inductor_SMD:L_0402_1005Metric, F.Cu at (23.3, 73.0)
- added R1: 27, Resistor_SMD:R_0402_1005Metric, F.Cu at (23.3, 77.0)
- added R15: 27, Resistor_SMD:R_0402_1005Metric, F.Cu at (26.2, 75.0)
- added R16: 33, Resistor_SMD:R_1206_3216Metric, F.Cu at (29.1, 82.9)
- added R19: 56k, Resistor_SMD:R_0402_1005Metric, F.Cu at (24.3, 32.5)
- added R2: 27, Resistor_SMD:R_0402_1005Metric, F.Cu at (26.2, 73.0)
- added R24: 9.1k, Resistor_SMD:R_0201_0603Metric, F.Cu at (73.2, 80.2)
- added R25: 9.1k, Resistor_SMD:R_0201_0603Metric, F.Cu at (73.2, 82.0)
- added R27: 33k, Resistor_SMD:R_0201_0603Metric, F.Cu at (73.2, 83.7)
- added R3: 33, Resistor_SMD:R_1206_3216Metric, F.Cu at (29.1, 79.6)
- added U4: LPS22DF, Package_LGA:ST_HLGA-10_2x2mm_P0.5mm_LayoutBorder3x2y, F.Cu at (76.4, 86.0)
- added Y2: 32MHz, Crystal:Crystal_SMD_3225-4Pin_3.2x2.5mm, F.Cu at (19.4, 22.3)
- J2: footprint Connector_PinHeader_2.54mm:PinHeader_2x04_P2.54mm_Vertical -> Connector_PinHeader_1.27mm:PinHeader_2x04_P1.27mm_Vertical
- moved IC1 104.6 mm to (68.7, 103.4), turned to 0 degrees
- moved IC2 94.9 mm to (74.2, 103.4), turned to 0 degrees
- moved J2 76.4 mm to (76.7, 89.8), turned to 0 degrees
- moved C29 72.8 mm to (21.1, 88.5), turned to 0 degrees
- moved SW2 69.7 mm to (72.4, 90.4), turned to 0 degrees
- moved IC5 68.8 mm to (36.0, 86.3), turned to 0 degrees
- moved SW1 62.7 mm to (67.8, 90.4), turned to 0 degrees
- moved IC9 54.9 mm to (67.4, 73.7), turned to 0 degrees
- moved AE1 46.1 mm to (6.75, 9.95), turned to 90 degrees
- moved U2 38.3 mm to (53.8, 15.7), turned to 90 degrees
- moved J1 32.9 mm to (43.5, 75.9), turned to 0 degrees
- moved IC6 32.4 mm to (15.1, 16.8), turned to -90 degrees
- moved Y1 30.7 mm to (49.3, 40.3)
- moved IC3 24.2 mm to (20.4, 28.5), turned to 0 degrees
- moved IC8 22.1 mm to (19.9, 16.8), turned to -90 degrees
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Connections:
- IC3 pad 19: /SCLK -> Net-(IC3-LNA_P)
- IC9 pad 8: /SCLK -> Net-(IC3-LNA_P)
- IC9 pad 9: /SCLK -> Net-(IC3-LNA_P)
- U1 pad 59: Net-(U1-ADC_AVDD) -> +3V3
- U1 pad 61: Net-(U1-ADC_AVDD) -> Net-(U1-VREG_AVDD)
- U3 pad 1: unconnected-(U3-RF_IN-Pad1) -> Net-(J6-Pin_1)
Routing:
- net GND: track 0.00 -> 61.0 mm, vias 0 -> 6
- net Net-(U1-GPIO26): track 0.00 -> 17.6 mm
- net Net-(U1-GPIO22): track 0.00 -> 16.2 mm
- net Net-(U1-GPIO31): track 0.00 -> 14.4 mm
- net Net-(IC3-RESET_N): track 0.00 -> 14.0 mm
- net Net-(U1-GPIO23): track 0.00 -> 13.4 mm
- net Net-(IC3-GPIO3): track 0.00 -> 13.3 mm
- net Net-(U1-GPIO24): track 0.00 -> 13.1 mm
- net Net-(IC3-GPIO2): track 0.00 -> 12.6 mm
- net Net-(IC1-AP_SCL_/_AP_SCLK): track 0.00 -> 12.1 mm
- net Net-(U1-GPIO29): track 0.00 -> 11.4 mm
- net Net-(U1-GPIO25): track 0.00 -> 11.2 mm
- net Net-(U1-GPIO2): track 0.00 -> 10.9 mm
- net Net-(U1-GPIO3): track 0.00 -> 10.4 mm
- net Net-(IC1-AP_SDA_/_AP_SDIO_/_AP_SDI): track 0.00 -> 10.4 mm
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- added copper zone on F.Cu, net Net-(AE1-A)
- added copper zone on F.Cu, net Net-(IC10-RF+_1)
- added copper zone on F.Cu, net Net-(IC10-RF-_1)
- added copper zone on F.Cu, net Net-(IC4-TR_SW)
- added copper zone on F.Cu, net Net-(IC8-RF+_1)
Other:
- board outline added: 70 x 50 mm

Commit message: pcb work
Parts:
- SW1: moved to B.Cu
- moved IC1 95.6 mm to (47.6, 10.2)
- moved IC2 95.5 mm to (65.5, 8.22)
- moved U4 87.3 mm to (34.2, 9.62)
- moved L3 71.2 mm to (59.5, 9.03), turned to 90 degrees
- moved L14 71.1 mm to (67.3, 11.8)
- moved R27 70.2 mm to (36.8, 23.7), turned to 180 degrees
- moved C8 69.4 mm to (56.1, 10.5), turned to 180 degrees
- moved R24 68.9 mm to (63.0, 12.1), turned to 180 degrees
- moved C7 68.8 mm to (65.8, 15.1), turned to -90 degrees
- moved C9 60.4 mm to (68.8, 8.00), turned to 180 degrees
- moved J3 56.6 mm to (48.2, 37.1)
- moved C6 53.7 mm to (63.0, 11.2), turned to 180 degrees
- moved IC5 52.1 mm to (41.5, 34.5), turned to 90 degrees
- moved J2 49.3 mm to (67.7, 41.2)
- moved SW1 48.5 mm to (48.4, 45.9), turned to 180 degrees
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Routing:
- net GND: track 61.0 -> 133.5 mm
- net Net-(U1-GPIO29): track 11.4 -> 50.1 mm, vias 0 -> 2
- net Net-(U1-GPIO31): track 14.4 -> 49.2 mm, vias 0 -> 2
- net Net-(IC4-HGM): track 0.00 -> 33.1 mm, vias 0 -> 2
- net Net-(IC4-LNA_EN): track 0.00 -> 31.8 mm, vias 0 -> 2
- net Net-(IC4-PA_EN): track 0.00 -> 26.6 mm, vias 0 -> 2
- net Net-(J10-Pin_3): track 0.00 -> 17.4 mm, vias 0 -> 1
- net Net-(U1-GPIO28): track 0.00 -> 16.4 mm, vias 0 -> 1
- net Net-(IC3-CSN): track 5.17 -> 19.5 mm
- net Net-(IC10-SDA): track 0.00 -> 12.8 mm, vias 0 -> 3
- net Net-(IC3-GPIO0): track 5.56 -> 16.5 mm
- net /MISO: track 5.64 -> 16.6 mm
- net Net-(U1-RUN): track 0.00 -> 8.58 mm
- net Net-(IC5-P0.0): track 0.00 -> 6.56 mm
- net Net-(J3-Pin_1): track 0.00 -> 6.05 mm
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- added copper zone on F.Cu, net +5V

Commit message: pcb work
Parts:
- moved R25 38.3 mm to (58.7, 46.5)
Routing:
- net Net-(IC3-GPIO2): track 12.6 -> 60.6 mm, vias 0 -> 4
- net Net-(IC3-RESET_N): track 14.0 -> 56.5 mm, vias 0 -> 4
- net Net-(IC3-GPIO3): track 13.3 -> 55.7 mm, vias 0 -> 4
- net Net-(IC3-GPIO0): track 16.5 -> 55.8 mm, vias 0 -> 2
- net /CS/PWM1: track 0.00 -> 18.5 mm, vias 0 -> 1
- net Net-(J9-Pin_3): track 0.00 -> 17.3 mm, vias 0 -> 1
- net Net-(IC3-CSN): track 19.5 -> 12.9 mm
- net /MISO: track 16.6 -> 12.8 mm
- net Net-(IC5-~{RESET}): track 0.00 -> 2.96 mm
- net Net-(U1-GPIO19): track 0.00 -> 2.61 mm
- net Net-(IC1-INT1_/_INT): track 0.00 -> 2.51 mm
- net Net-(U1-GPIO18): track 0.00 -> 2.38 mm
- net Net-(IC4-LNA_EN): track 31.8 -> 32.5 mm
- net GND: vias 6 -> 18

Commit message: pcb work
Parts:
- moved Y1 14.1 mm to (44.8, 27.6), turned to 0 degrees
Routing:
- net Net-(U1-GPIO3): track 10.4 -> 71.7 mm, vias 0 -> 2
- net Net-(U1-GPIO11): track 0.00 -> 8.71 mm, vias 0 -> 1
- net Net-(U1-GPIO10): track 0.00 -> 4.20 mm
- net Net-(U1-GPIO8): track 0.00 -> 3.84 mm
- net Net-(U1-GPIO9): track 0.00 -> 3.71 mm

Commit message: pcb work
Routing:
- net Net-(U1-GPIO2): track 10.9 -> 78.6 mm, vias 0 -> 2
- net Net-(U1-XOUT): track 0.00 -> 15.9 mm
- net Net-(U1-GPIO25): track 11.2 -> 12.0 mm
Changed lines of the file:
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@@
 	)
 	(segment
-		(start 9.473386 41.593698)
-		(end 10.25 41.593698)
-		(width 0.2)
-		(layer "F.Cu")
-		(net 83)
-	)
-	(segment
-		(start 9.227344 41.347656)
-		(end 9.473386 41.593698)
-		(width 0.2)
-		(layer "F.Cu")
-		(net 83)
-	)
-	(segment
-		(start 13.58815 39.51315)
+		(start 9.173944 41.994698)
+		(end 11.106602 41.994698)
+		(width 0.2)
+		(layer "F.Cu")
+		(net 83)
+	)
+	(segment
+		(start 8.362501 41.194698)
+		(end 8.373943 41.194698)
+		(width 0.2)
+		(layer "F.Cu")
+		(net 83)
+	)
+	(segment
+		(start 8.373943 41.194698)
+		(end 9.173944 41.994698)
+		(width 0.2)
+		(layer "F.Cu")
+		(net 83)
+	)
+	(segment
+		(start 11.106602 41.994698)
 		(end 14.95925 38.14205)
 		(width 0.2)
@@
 	)
 	(segment
-		(start 10.25 41.593698)
-		(end 11.507602 41.593698)
+		(start 8.362501 39.587498)
+		(end 8.362501 41.194698)
 		(width 0.2)
 		(layer "F.Cu")
@@
 	)
 	(segment
-		(start 8.362501 39.587498)
-		(end 8.362501 40.482813)
-		(width 0.2)
-		(layer "F.Cu")
-		(net 83)
-	)
-	(segment
-		(start 11.507602 41.593698)
-		(end 13.58815 39.51315)
-		(width 0.2)
-		(layer "F.Cu")
-		(net 83)
-	)
-	(segment
-		(start 8.362501 40.482813)
-		(end 9.227344 41.347656)
-		(width 0.2)
-		(layer "F.Cu")
-		(net 83)
+		(start 62.263069 35.455)
+		(end 61.613069 34.805)
+		(width 0.2)
+		(layer "F.Cu")
+		(net 84)
+	)
+	(segment
+		(start 10.09595 41.192698)
+		(end 9.639486 41.192698)
+		(width 0.2)
+		(layer "F.Cu")
+		(net 84)
+	)
+	(segment
+		(start 62.775 35.455)
+		(end 62.263069 35.455)
+		(width 0.2)
+		(layer "F.Cu")
+		(net 84)
+	)
+	(segment
+		(start 9.639486 41.192698)
+		(end 9.0125 40.565712)
+		(width 0.2)
+		(layer "F.Cu")
+		(net 84)
 	)
 	(segment
@@
 	)
 	(segment
-		(start 11.341502 41.192698)
-		(end 9.639486 41.192698)
-		(width 0.2)
-		(layer "F.Cu")
-		(net 84)
-	)
-	(segment
-		(start 9.639486 41.192698)
-		(end 9.0125 40.565712)
-		(width 0.2)
-		(layer "F.Cu")
-		(net 84)
-	)
-	(segment
-		(start 16.59215 39.20785)
-		(end 15.0613 37.677)
-		(width 0.2)
-		(layer "F.Cu")
-		(net 84)
-	)
-	(segment
-		(start 15.0613 37.677)
-		(end 14.8572 37.677)
-		(width 0.2)
-		(layer "F.Cu")
-		(net 84)
-	)
-	(segment
-		(start 14.8572 37.677)
-		(end 11.341502 41.192698)
-		(width 0.2)
-		(layer "F.Cu")
-		(net 84)
-	)
-	(segment
+		(start 10.39495 40.893698)
+		(end 10.09595 41.192698)
+		(width 0.2)
+		(layer "F.Cu")
+		(net 84)
+	)
+	(via
+		(at 9.94527 41.38768)
+		(size 0.6)
+		(drill 0.3)
+		(layers "F.Cu" "B.Cu")
+		(net 84)
+	)
+	(via
+		(at 61.613069 34.805)
+		(size 0.6)
+		(drill 0.3)
+		(layers "F.Cu" "B.Cu")
+		(net 84)
+	)
+	(segment
+		(start 63.376 43.1911)
+		(end 59.4861 47.081)
+		(width 0.2)
+		(layer "B.Cu")
+		(net 84)
+	)
+	(segment
+		(start 63.023943 33.649)
+		(end 63.376 34.001057)
+		(width 0.2)
+		(layer "B.Cu")
+		(net 84)
+	)
+	(segment
+		(start 10.007302 41.192698)
+		(end 10.025 41.175)
+		(width 0.2)
+		(layer "B.Cu")
+		(net 84)
+	)
+	(segment
+		(start 62.526057 33.649)
+		(end 63.023943 33.649)
+		(width 0.2)
+		(layer "B.Cu")
+		(net 84)
+	)
+	(segment
+		(start 59.4861 47.081)
+		(end 12.560359 47.081)
+		(width 0.2)
+		(layer "B.Cu")
+		(net 84)
+	)
+	(segment
+		(start 9.750288 41.192698)
+		(end 9.94527 41.38768)
+		(width 0.2)
+		(layer "B.Cu")
+		(net 84)
+	)
+	(segment
+		(start 7.524 42.044641)
+		(end 7.524 41.546755)
+		(width 0.2)
+		(layer "B.Cu")
+		(net 84)
+	)
+	(segment
+		(start 61.613069 34.561988)
+		(end 62.526057 33.649)
+		(width 0.2)
+		(layer "B.Cu")
+		(net 84)
+	)
+	(segment
+		(start 61.613069 34.805)
+		(end 61.613069 34.561988)
+		(width 0.2)
+		(layer "B.Cu")
+		(net 84)
+	)
+	(segment
+		(start 63.376 34.001057)
+		(end 63.376 43.1911)
+		(width 0.2)
+		(layer "B.Cu")
+		(net 84)
+	)
+	(segment
+		(start 7.878057 41.192698)
+		(end 9.750288 41.192698)
+		(width 0.2)
+		(layer "B.Cu")
+		(net 84)
+	)
+	(segment
+		(start 12.560359 47.081)
+		(end 7.524 42.044641)
+		(width 0.2)
+		(layer "B.Cu")
+		(net 84)
+	)
+	(segment
+		(start 7.524 41.546755)
+		(end 7.878057 41.192698)
+		(width 0.2)
+		(layer "B.Cu")
+		(net 84)
+	)
+	(segment
+		(start 52.33 39.055)
+		(end 41.5 28.225)
+		(width 0.2)
+		(layer "F.Cu")
+		(net 86)
+	)
+	(segment
+		(start 52.875 39.055)
+		(end 52.33 39.055)
+		(width 0.2)
+		(layer "F.Cu")
+		(net 86)
+	)
+	(segment

Commit message: pcb work
Parts:
- added C17: 4.7uF, Capacitor_SMD:C_0805_2012Metric, F.Cu at (65.4, 42.5)
- added C42: 4.7uF, Capacitor_SMD:C_0805_2012Metric, F.Cu at (64.8, 46.2)
- added R10: 1k, Resistor_SMD:R_0201_0603Metric, F.Cu at (68.8, 2.33)
- added R11: 1k, Resistor_SMD:R_0201_0603Metric, F.Cu at (44.9, 38.2)
- added R12: 1k, Resistor_SMD:R_0201_0603Metric, F.Cu at (46.0, 37.4)
- added R13: 1k, Resistor_SMD:R_0201_0603Metric, F.Cu at (43.7, 44.2)
- added R14: 1k, Resistor_SMD:R_0201_0603Metric, F.Cu at (36.2, 29.8)
- added R17: 1k, Resistor_SMD:R_0201_0603Metric, F.Cu at (43.7, 42.7)
- added R18: 1k, Resistor_SMD:R_0201_0603Metric, F.Cu at (43.7, 43.5)
- added R20: 1k, Resistor_SMD:R_0201_0603Metric, F.Cu at (61.6, 45.4)
- added R21: 1k, Resistor_SMD:R_0201_0603Metric, F.Cu at (61.6, 46.1)
- added R22: 1k, Resistor_SMD:R_0201_0603Metric, F.Cu at (61.0, 48.5)
- added R26: 1k, Resistor_SMD:R_0201_0603Metric, F.Cu at (58.6, 47.3)
- added R4: 1k, Resistor_SMD:R_0201_0603Metric, F.Cu at (67.2, 35.3)
- added R5: 1k, Resistor_SMD:R_0201_0603Metric, F.Cu at (41.6, 45.5)
- added R6: 1k, Resistor_SMD:R_0201_0603Metric, F.Cu at (61.6, 7.87)
- added R7: 1k, Resistor_SMD:R_0201_0603Metric, F.Cu at (61.6, 9.32)
- added R8: 1k, Resistor_SMD:R_0201_0603Metric, F.Cu at (67.7, 1.20)
- added R9: 1k, Resistor_SMD:R_0201_0603Metric, F.Cu at (67.7, 1.95)
- moved C31 87.3 mm to (6.25, 21.4), turned to 90 degrees
- moved C30 83.8 mm to (6.28, 25.0), turned to -90 degrees
- moved C32 83.5 mm to (5.47, 29.9)
- moved C36 80.7 mm to (3.42, 41.0)
- moved C35 76.5 mm to (70.2, 7.25)
- moved C21 75.6 mm to (70.2, 8.15)
- moved C37 75.3 mm to (70.1, 9.78)
- moved L11 72.5 mm to (30.2, 20.1)
- moved C41 66.3 mm to (36.3, 30.6)
- moved C39 63.7 mm to (70.1, 11.9)
- moved R1 62.5 mm to (68.0, 33.2), turned to -90 degrees
- moved L1 61.9 mm to (67.5, 41.5), turned to -90 degrees
- moved J1 58.7 mm to (68.4, 22.7)
- moved R2 58.4 mm to (68.9, 33.2), turned to 90 degrees
- moved IC9 58.2 mm to (26.5, 32.3), turned to 90 degrees
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Connections:
- C34 pad 1: unconnected-(C34-Pad1) -> GND
- C34 pad 2: unconnected-(C34-Pad2) -> +3V3
- U2 pad 6: (no net) -> GND
- U2 pad 7: (no net) -> GND
Routing:
- net GND: track 133.5 -> 458.4 mm, vias 18 -> 41
- net +3V3: track 14.1 -> 170.3 mm, vias 0 -> 32
- net +5V: track 0.83 -> 140.0 mm, vias 1 -> 3
- net /MISO: track 12.8 -> 139.7 mm, vias 0 -> 4
- net /SCLK: track 8.13 -> 132.6 mm, vias 0 -> 5
- net /MOSI: track 6.75 -> 131.2 mm, vias 0 -> 6
- net Net-(IC1-AP_SCL_/_AP_SCLK): track 12.1 -> 123.0 mm, vias 0 -> 4
- net Net-(IC2-EN1): track 0.00 -> 102.6 mm, vias 0 -> 2
- net Net-(IC1-AP_SDA_/_AP_SDIO_/_AP_SDI): track 10.4 -> 111.7 mm, vias 0 -> 4
- net +BATT: track 0.00 -> 99.6 mm, vias 0 -> 3
- net Net-(J4-Pin_9): track 0.00 -> 98.9 mm, vias 0 -> 2
- net Net-(J4-Pin_5): track 0.00 -> 82.1 mm, vias 0 -> 1
- net Net-(J4-Pin_7): track 0.00 -> 74.5 mm, vias 0 -> 1
- net /CS/PWM1: track 18.5 -> 92.8 mm
- net Net-(J4-Pin_6): track 0.00 -> 73.0 mm, vias 0 -> 2
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- added copper zone on F.Cu, net +1V1
- added copper zone on F.Cu, net +3V3
- added copper zone on In1.Cu, net +3V3
- added copper zone on F.Cu, net GND
- added copper zone on In2.Cu, net GND
- added copper zone on F.Cu, net Net-(C41-Pad1)
- added copper zone on F.Cu, net Net-(IC3-LNA_P)
- added copper zone on F.Cu, net Net-(IC4-PA_IN)
Other:
- board size 70 x 50 mm -> 75 x 50 mm

Commit message: pcb work final
Parts:
- moved C32 3.12 mm to (6.28, 26.9), turned to 90 degrees
- moved R1 1.43 mm to (66.5, 33.1)
- moved R2 1.05 mm to (67.9, 33.1)
Routing:
- net +1V1: track 10.8 -> 41.8 mm, vias 0 -> 3
- net Net-(IC10-SCL): track 31.5 -> 56.4 mm, vias 2 -> 6
- net Net-(U1-USB_DM): track 0.00 -> 16.0 mm, vias 0 -> 2
- net Net-(U1-USB_DP): track 0.00 -> 15.8 mm, vias 0 -> 2
- net GND: track 458.4 -> 466.2 mm, vias 41 -> 45
- net Net-(IC2-EN1): track 102.6 -> 95.1 mm
- net Net-(J4-Pin_9): track 98.9 -> 103.0 mm
- net Net-(J1-Pin_2): track 6.37 -> 9.79 mm, vias 0 -> 1
- net +3V3: track 170.3 -> 172.8 mm, vias 32 -> 33
- net Net-(J1-Pin_3): track 3.49 -> 5.81 mm, vias 0 -> 1
- net +5V: track 140.0 -> 140.6 mm

Commit message: pcb work
Parts:
- moved C27 0.12 mm to (21.8, 24.3)
- moved Y2 0.07 mm to (19.3, 22.2)
- moved C25 0.07 mm to (16.8, 22.2)
- moved C10 0.06 mm to (23.1, 25.1)
- moved C24 0.05 mm to (21.9, 22.2)
Routing:
- net +3V3: track 172.8 -> 494.8 mm, vias 33 -> 37
- net GND: track 466.2 -> 774.1 mm, vias 45 -> 49
- net Net-(IC10-SDA): track 20.2 -> 93.4 mm, vias 4 -> 7
- net Net-(IC10-SCL): track 56.4 -> 95.3 mm, vias 6 -> 8
- net Net-(IC5-P1.6): track 15.9 -> 33.9 mm, vias 2 -> 3
- net +1V8: track 73.3 -> 79.7 mm
- net Net-(J4-Pin_8): track 72.1 -> 76.5 mm
- net Net-(IC10-RF-_1): track 4.48 -> 6.99 mm
- net /SCLK: track 132.6 -> 135.0 mm
- net Net-(IC3-LNA_P): track 5.44 -> 7.38 mm
- net Net-(IC5-P1.1): track 19.8 -> 21.8 mm
- net Net-(IC1-AP_SDA_/_AP_SDIO_/_AP_SDI): track 111.7 -> 113.6 mm
- net Net-(J7-Pin_3): track 64.9 -> 63.4 mm
- net /MOSI: track 131.2 -> 132.6 mm
- net Net-(J4-Pin_7): track 74.5 -> 75.9 mm
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