File: hardware/main/main.kicad_pcb (KiCad board)
At the start: 4 copper layers, 75 x 50 mm, 112 parts, among them IC1 ICM-42688-P, IC10 PE64906B-Z, IC2 PAM2306DYPAA, IC3 CC1121RHBR, IC4 CC1190RGVR, IC5 TXE8116DGSR, IC6 PE64906B-Z, IC7 PE64906B-Z, IC8 PE64906B-Z, IC9 PE64906B-Z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

Commit message: hardware edits mainly
Routing:
- net GND: track 774.1 -> 777.3 mm, vias 49 -> 50
- added copper zone on B.Cu, net +3V3

Commit message: pcb fixes
Parts:
- moved C3 0.16 mm to (73.1, 43.2)
- moved C26 0.05 mm to (20.1, 24.7)
Connections:
- IC1 pad 1: unconnected-(IC1-AP_SDO_/_AP_AD0-Pad1) -> GND
- IC10 pad 6: Net-(IC10-SCL) -> Net-(IC10-SEN)
- IC3 pad 7: /SCLK -> /MOSI
- IC3 pad 8: /MOSI -> /SCLK
- IC5 pad 22: /MOSI -> /SCLK
- IC5 pad 23: /SCLK -> /MOSI
- U1 pad 68: +5V -> +3V3
- U3 pad 29: Net-(IC1-AP_SDA_/_AP_SDIO_/_AP_SDI) -> Net-(IC1-AP_SCL_/_AP_SCLK)
- U3 pad 30: Net-(IC1-AP_SCL_/_AP_SCLK) -> Net-(IC1-AP_SDA_/_AP_SDIO_/_AP_SDI)
Routing:
- net GND: track 777.3 -> 873.8 mm, vias 50 -> 55
- net +5V: track 140.6 -> 116.1 mm, vias 3 -> 2
- net +3V3: track 494.8 -> 499.0 mm
- net Net-(IC1-AP_SDA_/_AP_SDIO_/_AP_SDI): track 113.6 -> 117.0 mm
- net Net-(IC10-SCL): track 95.3 -> 92.5 mm
- net /MOSI: track 132.6 -> 135.0 mm, vias 6 -> 8
- net Net-(IC1-AP_SCL_/_AP_SCLK): track 123.0 -> 124.2 mm
- net Net-(U1-GPIO9): track 23.3 -> 24.2 mm
- net Net-(U1-GPIO11): track 20.2 -> 19.6 mm
