File: hardware/esc/esc/esc.kicad_pcb (KiCad board)
At the start: 4 copper layers, 298 parts, among them IC1 IR2136SPBF, IC2 IR2136SPBF, IC3 IR2136SPBF, IC4 IR2136SPBF, IC5 IR2136SPBF, IC6 IR2136SPBF, IC7 TLA2528IRTER, IC8 MP9486AGN-Z, J1 USB-C, J10 GPIO, J11 Conn_01x08_Pin, J2 DEBUG, J3 TEMP-GPIO, Q1 NMOS, Q10 NMOS, Q11 NMOS, Q12 NMOS, Q13 NMOS, Q14 NMOS, Q15 NMOS, Q16 NMOS, Q17 NMOS, Q18 NMOS, Q19 NMOS, Q2 NMOS, Q20 NMOS, Q21 NMOS, Q22 NMOS, Q23 NMOS, Q24 NMOS, Q25 NMOS, Q26 NMOS, Q27 NMOS, Q28 NMOS, Q29 NMOS, Q3 NMOS, Q30 NMOS, Q31 NMOS, Q32 NMOS, Q33 NMOS, Q34 NMOS, Q35 NMOS, Q36 NMOS, Q4 NMOS, Q5 NMOS, Q6 NMOS, Q7 NMOS, Q8 NMOS, Q9 NMOS, SW1 SW_Push, SW2 SW_Push, U1 RP2354B, U10 INA240A2PW, U11 INA240A2PW, U12 INA240A2PW, U14 TMP110D, U15 TMP110D, U16 AZ1117CH2-3.3, U2 INA240A2PW, U3 INA240A2PW, U4 INA240A2PW, U5 INA240A2PW, U6 INA240A2PW, U7 INA240A2PW, U8 INA240A2PW, U9 INA240A2PW, Y1 12MHz

Commit message: Auto-sync ESC PCB 2026-05-09 17:28:29
Parts:
- removed C51, C64, C75, C84, C85, C88, C91: 4.7uF, Capacitor_SMD:CP_Elec_6.3x7.7
- removed R56, R57: SHUNT, Fuse:Fuse_1206_3216Metric_Pad1.42x1.75mm_HandSolder
- removed U7: INA240A2PW, Package_SO:TSSOP-8_4.4x3mm_P0.65mm
- added Q37: SMALL, Package_TO_SOT_SMD:SOT-23-3, F.Cu at (117.1, 77.6)
- added Q38: SMALL, Package_TO_SOT_SMD:SOT-23-3, F.Cu at (8.80, 23.5)
- C1, C10, C11, C16, C17, C18, C23, C24, C25, C3, C30, C31, C32, C39, C40, C41, C44, C45, C5, C9: footprint Capacitor_SMD:CP_Elec_6.3x7.7 -> Capacitor_SMD:C_1206_3216Metric
- C43, C46, C50, C57: value 4.7uF -> 1uF; footprint Capacitor_SMD:CP_Elec_6.3x7.7 -> Capacitor_SMD:C_0402_1005Metric
- C48, C54, C55, C58, C61, C63, C66, C71, C72, C73, C74, C76: value 4.7uF -> 10uF; footprint Capacitor_SMD:CP_Elec_6.3x7.7 -> Capacitor_SMD:C_0402_1005Metric
- C60, C67: value 4.7uF -> 0.1uF; footprint Capacitor_SMD:CP_Elec_6.3x7.7 -> Capacitor_SMD:C_0603_1608Metric
- R55: value SHUNT -> 1k; footprint Fuse:Fuse_1206_3216Metric_Pad1.42x1.75mm_HandSolder -> Resistor_SMD:R_0201_0603Metric
- moved U15 262.9 mm to (5.62, 24.9)
- moved D14 246.8 mm to (3.45, 20.1), turned to 180 degrees
- moved R54 245.7 mm to (6.59, 17.4), turned to 180 degrees
- moved R52 236.7 mm to (22.1, 14.5), turned to 90 degrees
- moved IC1 229.3 mm to (62.2, 32.3)
- moved TP22 227.0 mm to (2.85, 28.1), turned to 90 degrees
- moved TP16 226.5 mm to (9.49, 2.49)
- moved C35 225.5 mm to (6.50, 15.9), turned to 180 degrees
- moved Q26 224.4 mm to (4.05, 8.41)
- moved R53 222.4 mm to (36.6, 21.3), turned to 180 degrees
- moved C29 221.9 mm to (30.0, 42.3)
- moved D13 221.6 mm to (29.4, 19.5)
- moved TP21 219.7 mm to (8.33, 28.0), turned to 180 degrees
- moved TP17 217.2 mm to (23.8, 2.47), turned to -90 degrees
- moved TP20 216.0 mm to (8.33, 33.1), turned to 180 degrees
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Connections:
- C17 pad 1: Net-(IC3-VB1) -> Net-(IC3-VS1)
- C17 pad 2: Net-(IC3-VS1) -> Net-(IC3-VB1)
- C40 pad 1: Net-(IC6-VB1) -> Net-(IC6-VS1)
- C40 pad 2: Net-(IC6-VS1) -> Net-(IC6-VB1)
- C60 pad 1: +3V3 -> GND
- C60 pad 2: GND -> +5V
- C63 pad 1: +3V3 -> +5V
- C66 pad 1: +3V3 -> +5V
- C67 pad 1: +3V3 -> GND
- C67 pad 2: GND -> +5V
- C73 pad 1: +5V -> GND
- C73 pad 2: GND -> +1V1
- C76 pad 1: +5V -> GND
- C76 pad 2: GND -> +5V
- C77 pad 1: Net-(U16-GND) -> GND
- IC5 pad 9: Net-(IC5-ITRIP) -> unconnected-(IC5-ITRIP-Pad9)
- R55 pad 1: GND -> Net-(IC8-DIM)
- R55 pad 2: Net-(U7-+) -> GND
- R64 pad 1: Net-(U7-+) -> GND
- R65 pad 1: Net-(U7-+) -> GND
- R66 pad 1: Net-(U7-+) -> GND
- R67 pad 1: Net-(U7-+) -> GND
- R68 pad 1: Net-(U7-+) -> GND
- R69 pad 1: Net-(U7-+) -> GND
- R70 pad 1: Net-(U7-+) -> GND
- R71 pad 1: Net-(U7-+) -> GND
- R72 pad 1: Net-(U7-+) -> GND
- U1 pad 13: Net-(U1-GPIO14) -> Net-(Q37-G)
- U1 pad 14: Net-(U1-GPIO15) -> Net-(Q38-G)
- U14 pad 3: Net-(U1-GPIO14) -> Net-(Q37-D)
- U14 pad 5: +3V3 -> Net-(Q37-D)
- U15 pad 3: Net-(U1-GPIO15) -> Net-(Q38-D)
- U15 pad 5: +3V3 -> Net-(Q38-D)
- U16 pad 2: Net-(U16-GND) -> GND
Routing:
- net GND: track 2.62 -> 772.5 mm, vias 0 -> 672
- net +3V3: track 34.8 -> 577.9 mm, vias 3 -> 47
- net Net-(IC7-SDA): track 0.00 -> 186.9 mm, vias 0 -> 9
- net Net-(IC1-~{HIN3}): track 0.00 -> 155.0 mm, vias 0 -> 7
- net Net-(IC1-~{LIN3}): track 0.00 -> 153.9 mm, vias 0 -> 7
- net Net-(IC7-SCL): track 0.00 -> 144.7 mm, vias 0 -> 5
- net Net-(IC1-~{LIN1}): track 0.00 -> 137.8 mm, vias 0 -> 5
- net Net-(IC1-~{LIN2}): track 0.00 -> 124.8 mm, vias 0 -> 5
- net Net-(IC1-~{HIN1}): track 0.00 -> 116.3 mm, vias 0 -> 6
- net Net-(IC1-~{HIN2}): track 0.00 -> 114.6 mm, vias 0 -> 6
- net Net-(IC7-ADDR): track 0.00 -> 107.5 mm, vias 0 -> 3
- net Net-(IC3-~{HIN2}): track 0.00 -> 102.2 mm, vias 0 -> 4
- net Net-(IC3-~{HIN1}): track 0.00 -> 95.6 mm, vias 0 -> 4
- net Net-(IC2-ITRIP): track 16.2 -> 109.9 mm, vias 0 -> 5
- net Net-(IC4-ITRIP): track 0.00 -> 90.3 mm, vias 0 -> 4
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- added copper zone on In2.Cu, net +3V3
- added copper zone on In1.Cu, net +5V
- added copper zone on F.Cu, net +BATT
- added copper zone on In2.Cu, net +BATT
- added copper zone on B.Cu, net GND
- added copper zone on F.Cu, net GND
- added copper zone on F.Cu, net Net-(IC1-VS1)
- added copper zone on F.Cu, net Net-(IC1-VS2)
- added copper zone on F.Cu, net Net-(IC1-VS3)
- added copper zone on F.Cu, net Net-(IC2-VS1)
- added copper zone on F.Cu, net Net-(IC2-VS2)
- added copper zone on F.Cu, net Net-(IC2-VS3)
- added copper zone on F.Cu, net Net-(IC3-VS1)
- added copper zone on F.Cu, net Net-(IC3-VS2)
- added copper zone on F.Cu, net Net-(IC3-VS3)
- added copper zone on F.Cu, net Net-(IC4-VS1)
- added copper zone on F.Cu, net Net-(IC4-VS2)
- added copper zone on F.Cu, net Net-(IC4-VS3)
- added copper zone on F.Cu, net Net-(IC5-VS1)
- added copper zone on F.Cu, net Net-(IC5-VS2)
- added copper zone on F.Cu, net Net-(IC5-VS3)
- added copper zone on F.Cu, net Net-(IC6-VS1)
- added copper zone on F.Cu, net Net-(IC6-VS2)
- added copper zone on F.Cu, net Net-(IC6-VS3)
- added copper zone on F.Cu, net Net-(U10-+)
- added copper zone on In1.Cu, net Net-(U10-+)
- added copper zone on F.Cu, net Net-(U11-+)
- added copper zone on In1.Cu, net Net-(U11-+)
- added copper zone on F.Cu, net Net-(U12-+)
- added copper zone on In1.Cu, net Net-(U12-+)
- added copper zone on F.Cu, net Net-(U2-+)
- added copper zone on In1.Cu, net Net-(U2-+)
- added copper zone on F.Cu, net Net-(U3-+)
- added copper zone on In1.Cu, net Net-(U3-+)
- added copper zone on F.Cu, net Net-(U4-+)
- added copper zone on In1.Cu, net Net-(U4-+)
- added copper zone on F.Cu, net Net-(U5-+)
- added copper zone on In1.Cu, net Net-(U5-+)
- added copper zone on F.Cu, net Net-(U6-+)
- added copper zone on In1.Cu, net Net-(U6-+)
- added copper zone on F.Cu, net Net-(U8-+)
- added copper zone on In1.Cu, net Net-(U8-+)
- added copper zone on F.Cu, net Net-(U9-+)
- added copper zone on In1.Cu, net Net-(U9-+)
Other:
- board outline added: 120 x 80 mm

Commit message: Auto-sync ESC PCB 2026-05-09 18:43:14
Routing:
- net Net-(Q37-G): track 63.0 -> 116.6 mm, vias 2 -> 5

Commit message: Auto-sync ESC PCB 2026-05-09 23:58:51
Parts:
- moved C66 102.6 mm to (88.1, 23.4), turned to -90 degrees
- moved C67 100.9 mm to (86.8, 23.5), turned to 90 degrees
- moved C60 99.1 mm to (85.2, 23.5), turned to 90 degrees
- moved C63 97.6 mm to (84.0, 23.4), turned to -90 degrees
- moved C76 96.4 mm to (83.0, 23.5), turned to 90 degrees
- moved C71 94.9 mm to (81.8, 23.4), turned to -90 degrees
- moved R95 83.8 mm to (41.6, 20.2), turned to 0 degrees
Routing:
- net +3V3: track 577.9 -> 654.0 mm, vias 47 -> 51
- net Net-(IC7-SCL): track 144.7 -> 200.5 mm, vias 5 -> 6
- net Net-(U1-VREG_AVDD): track 0.43 -> 29.3 mm, vias 1 -> 3
- net +BATT: track 47.8 -> 57.2 mm, vias 539 -> 540
- net +5V: track 74.9 -> 82.5 mm, vias 21 -> 22
- net GND: track 772.5 -> 778.8 mm
- net Net-(IC4-LO3): track 51.9 -> 53.6 mm
- net Net-(Q37-G): track 116.6 -> 118.3 mm
- net Net-(IC7-SDA): track 186.9 -> 188.5 mm
- net Net-(U1-GPIO44/ADC4): track 44.7 -> 43.8 mm
- net Net-(IC5-VB2): track 33.3 -> 34.0 mm
- net Net-(IC1-VB1): track 52.5 -> 51.8 mm
