File: hardware/esc/esc/bec.kicad_sch (KiCad schematic)
At the start: 31 parts, among them IC1 LM5148QRGYRQ1, IC2 LM5148QRGYRQ1, Q1 NX138AKHH, Q2 BUK9K12-80LX, Q3 BUK9K12-80LX, Q4 NX138AKHH

Commit message: more pcb stuff
Parts:
- added R?: 71.4k, Resistor_SMD:R_0402_1005Metric, symbol Device:R_Small
- added R?: 90.9k, Resistor_SMD:R_0402_1005Metric, symbol Device:R_Small
- renumbered C9 to C?, C12 to C?, C4 to C?, C6 to C?, C8 to C?, C11 to C?, C2 to C?, C10 to C?, C3 to C?, C7 to C?, C5 to C?, C1 to C?, D1 to D?, D2 to D?, IC2 to IC?, IC1 to IC?, L2 to L?, L1 to L?, Q1 to Q?, Q3 to Q?, Q4 to Q?, Q2 to Q?, R1 to R?, R5 to R?, R6 to R?, R7 to R?, R8 to R?, R4 to R?, R10 to R?, R3 to R?, R2 to R?
Connections:
- net BEC_SHDN: no longer Q?.1 (G)
- net GND: now also R?.1, R?.1
- net at IC?.3 (CNFG): now also R?.2 (x2)
- new net BEC_SHDN2: Q?.1 (G)
- no-connect marks 14 -> 12

Commit message: more pcb stuff
Parts:
- IC1, IC2: renamed from IC?; footprint LM5148QRGYRQ1 -> LM5148QRGYRQ1:LM5148QRGYRQ1
- L1, L2: renamed from L?; footprint Inductor_SMD:L_APV_APH1770 -> Connector_PinHeader_2.54mm:PinHeader_1x02_P2.54mm_Vertical
- Q1, Q4: renamed from Q?; footprint NX138AKHH -> NX138AKH:NX138AKHH
- Q2, Q3: renamed from Q?; footprint BUK7K6R840E115 -> BUK9K12-80L:BUK7K6R840E115
- gave numbers to parts that had none: 25
Connections:
- net at IC2.17 (PG/SYNCOUT): now also IC1.18 (PFM/SYNC)
