File: hardware/esc/esc/esc.kicad_sch (KiCad schematic)
At the start: 298 parts, among them IC1 IR2136SPBF, IC2 IR2136SPBF, IC3 IR2136SPBF, IC4 IR2136SPBF, IC5 IR2136SPBF, IC6 IR2136SPBF, IC7 TLA2528IRTER, IC8 MP9486AGN-Z, J1 USB-C, J10 GPIO, J11 Conn_01x08_Pin, J2 DEBUG, J3 TEMP-GPIO, Q1 NMOS, Q10 NMOS, Q11 NMOS, Q12 NMOS, Q13 NMOS, Q14 NMOS, Q15 NMOS, Q16 NMOS, Q17 NMOS, Q18 NMOS, Q19 NMOS, Q2 NMOS, Q20 NMOS, Q21 NMOS, Q22 NMOS, Q23 NMOS, Q24 NMOS, Q25 NMOS, Q26 NMOS, Q27 NMOS, Q28 NMOS, Q29 NMOS, Q3 NMOS, Q30 NMOS, Q31 NMOS, Q32 NMOS, Q33 NMOS, Q34 NMOS, Q35 NMOS, Q36 NMOS, Q4 NMOS, Q5 NMOS, Q6 NMOS, Q7 NMOS, Q8 NMOS, Q9 NMOS, SW1 SW_Push, SW2 SW_Push, U1 RP2354B, U10 INA240A2PW, U11 INA240A2PW, U12 INA240A2PW, U14 TMP110D, U15 TMP110D, U16 AZ1117CH2-3.3, U2 INA240A2PW, U3 INA240A2PW, U4 INA240A2PW, U5 INA240A2PW, U6 INA240A2PW, U7 INA240A2PW, U8 INA240A2PW, U9 INA240A2PW, Y1 12MHz

Commit message: pcbss
Other:
- added sheet BEC (bec.kicad_sch)

Commit message: more pcb stuff
Connections:
- net BEC_SHDN: now also IC7.6 (AIN7/GPIO7), J3.8 (Pin_8)
- net BEC_SHDN2: now reaches IC7.5 (AIN6/GPIO6), J3.7 (Pin_7)
Other:
- sheet BEC ports: added BEC_SHDN2; removed none
Changed lines of the file:
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@@
 	(wire
 		(pts
-			(xy 31.75 346.71) (xy 39.37 346.71)
+			(xy 101.6 363.22) (xy 93.98 363.22)
 		)
 		(stroke
@@
 	(wire
 		(pts
-			(xy 29.21 328.93) (xy 39.37 328.93)
+			(xy 106.68 381) (xy 93.98 381)
 		)
 		(stroke
@@
 	(wire
 		(pts
-			(xy 138.43 374.65) (xy 138.43 372.11)
+			(xy 138.43 375.92) (xy 138.43 372.11)
 		)
 		(stroke
@@
 	(wire
 		(pts
-			(xy 123.19 374.65) (xy 138.43 374.65)
+			(xy 123.19 375.92) (xy 138.43 375.92)
 		)
 		(stroke
@@
 	(wire
 		(pts
+			(xy 93.98 375.92) (xy 104.14 375.92)
+		)
+		(stroke
+			(width 0)
+			(type default)
+		)
+	)
+	(wire
+		(pts
 			(xy 76.2 52.07) (xy 86.36 52.07)
 		)
@@
 	(wire
 		(pts
-			(xy 54.61 319.405) (xy 54.61 317.5)
+			(xy 78.74 390.525) (xy 78.74 392.43)
 		)
 		(stroke
@@
 	(wire
 		(pts
-			(xy 123.19 354.33) (xy 123.19 374.65)
+			(xy 123.19 354.33) (xy 123.19 375.92)
 		)
 		(stroke
@@
 	(wire
 		(pts
-			(xy 31.75 322.58) (xy 39.37 322.58)
+			(xy 101.6 387.35) (xy 93.98 387.35)
 		)
 		(stroke
@@
 		)
 	)
+	(label "BEC_SHDN2"
+		(at 124.46 372.11 0)
+		(effects
+			(font
+				(size 1.27 1.27)
+			)
+			(justify left bottom)
+		)
+	)
+	(label "BEC_SHDN"
+		(at 129.54 375.92 0)
+		(effects
+			(font
+				(size 1.27 1.27)
+			)
+		)
+	)
+	(label "BEC_SHDN2"
+		(at 104.14 375.92 0)
+		(effects
+			(font
+				(size 1.27 1.27)
+			)
+			(justify left bottom)
+		)
+	)
 	(label "BEC_SHDN"
-		(at 29.21 328.93 0)
+		(at 106.68 381 0)
 		(effects
 			(font
@@
 	(symbol
 		(lib_id "power:+BATT")
-		(at 31.75 322.58 0)
+		(at 101.6 387.35 180)
 		(unit 1)
 		(exclude_from_sim no)
@@
 		(dnp no)
 		(property "Reference" "#PWR0145"
-			(at 31.75 326.39 0)
+			(at 101.6 383.54 0)
 			(effects
 				(font
@@
 		)
 		(property "Value" "+BATT"
-			(at 31.75 317.5 0)
+			(at 101.6 392.43 0)
 			(effects
 				(font
@@
 		)
 		(property "Footprint" ""
-			(at 31.75 322.58 0)
+			(at 101.6 387.35 0)
 			(effects
 				(font
@@
 		)
 		(property "Datasheet" ""
-			(at 31.75 322.58 0)
+			(at 101.6 387.35 0)
 			(effects
 				(font
@@
 		)
 		(property "Description" "Power symbol creates a global label with name \"+BATT\""
-			(at 31.75 322.58 0)
+			(at 101.6 387.35 0)
 			(effects
 				(font
@@
 	(symbol
 		(lib_id "power:+5V")
-		(at 54.61 317.5 0)
+		(at 78.74 392.43 180)
 		(unit 1)
 		(exclude_from_sim no)
@@
 		(dnp no)
 		(property "Reference" "#PWR0146"
-			(at 54.61 321.31 0)
+			(at 78.74 388.62 0)
 			(effects
 				(font
@@
 		)
 		(property "Value" "+5V"
-			(at 54.61 313.69 0)
+			(at 78.74 396.24 0)
 			(effects
 				(font
@@
 		)
 		(property "Footprint" ""
-			(at 54.61 317.5 0)
+			(at 78.74 392.43 0)
 			(effects
 				(font
@@
 		)
 		(property "Datasheet" ""
-			(at 54.61 317.5 0)
+			(at 78.74 392.43 0)
 			(effects
 				(font
@@
 		)
 		(property "Description" "Power symbol creates a global label with name \"+5V\""
-			(at 54.61 317.5 0)
+			(at 78.74 392.43 0)
 			(effects
 				(font
@@
 	(symbol
 		(lib_id "power:GND")
-		(at 31.75 346.71 180)
+		(at 101.6 363.22 0)
 		(unit 1)
 		(exclude_from_sim no)
@@
 		(dnp no)
 		(property "Reference" "#PWR0147"
-			(at 31.75 340.36 0)
+			(at 101.6 369.57 0)
 			(effects
 				(font
@@
 		)
 		(property "Value" "GND"
-			(at 31.75 341.63 0)
+			(at 101.6 368.3 0)
 			(effects
 				(font
@@
 		)
 		(property "Footprint" ""
-			(at 31.75 346.71 0)
+			(at 101.6 363.22 0)
 			(effects
 				(font
@@
 		)
 		(property "Datasheet" ""
-			(at 31.75 346.71 0)
+			(at 101.6 363.22 0)
 			(effects
 				(font
@@
 		)
 		(property "Description" "Power symbol creates a global label with name \"GND\" , ground"
-			(at 31.75 346.71 0)
+			(at 101.6 363.22 0)
 			(effects
 				(font
@@
 	)
 	(sheet
-		(at 39.37 319.405)
-		(size 24.13 31.75)
+		(at 74.93 360.045)
+		(size 19.05 30.48)
 		(exclude_from_sim no)
 		(in_bom yes)
@@
 		)
 		(property "Sheetname" "BEC"
-			(at 39.37 318.6934 0)
+			(at 74.93 359.3334 0)
 			(effects
 				(font
@@
 		)
 		(property "Sheetfile" "bec.kicad_sch"
-			(at 39.37 351.7396 0)
+			(at 74.93 391.1096 0)
 			(effects
 				(font
@@
 		)
 		(pin "BATT_IN" input
-			(at 39.37 322.58 180)
+			(at 93.98 387.35 0)
 			(effects
 				(font
 					(size 1.27 1.27)
 				)
-				(justify left)
+				(justify right)
 			)
 		)
 		(pin "BEC_5V" output
-			(at 54.61 319.405 90)
+			(at 78.74 390.525 270)
+			(effects
+				(font
+					(size 1.27 1.27)
+				)
+				(justify left)
+			)
+		)
+		(pin "BEC_SHDN" input
+			(at 93.98 381 0)
 			(effects
 				(font
@@
 			)
 		)
-		(pin "GND" passive
-			(at 39.37 346.71 180)
+		(pin "BEC_SHDN2" input
+			(at 93.98 375.92 0)
 			(effects
 				(font
 					(size 1.27 1.27)
 				)
-				(justify left)
+				(justify right)
 			)
 		)
-		(pin "BEC_SHDN" input
-			(at 39.37 328.93 180)
+		(pin "GND" passive
+			(at 93.98 363.22 0)
 			(effects
 				(font
 					(size 1.27 1.27)
 				)
-				(justify left)
+				(justify right)
 			)
 		)

Commit message: more pcb stuff
Parts:
- removed C1, C11, C18: 4.7uF, Capacitor_SMD:CP_Elec_6.3x7.7, symbol Device:C_Small
- removed R55, R56, R57: SHUNT, Fuse:Fuse_1206_3216Metric_Pad1.42x1.75mm_HandSolder, symbol Device:R_Small
- removed U7: INA240A2PW, Package_SO:TSSOP-8_4.4x3mm_P0.65mm, symbol Amplifier_Current:INA240A2PW
- C1: renamed from C85; footprint Capacitor_SMD:CP_Elec_6.3x7.7 -> Capacitor_SMD:C_0402_1005Metric
- C10: renamed from C84; footprint Capacitor_SMD:CP_Elec_6.3x7.7 -> Capacitor_SMD:C_0402_1005Metric
- C11: renamed from C88; footprint Capacitor_SMD:CP_Elec_6.3x7.7 -> Capacitor_SMD:C_0402_1005Metric
- C16: renamed from C48; footprint Capacitor_SMD:CP_Elec_6.3x7.7 -> Capacitor_SMD:C_0402_1005Metric
- C19: renamed from C45; footprint Capacitor_SMD:CP_Elec_6.3x7.7 -> Capacitor_SMD:C_0402_1005Metric
- C2: renamed from C91; footprint Capacitor_SMD:CP_Elec_6.3x7.7 -> Capacitor_SMD:C_0402_1005Metric
- C20: renamed from C44; footprint Capacitor_SMD:CP_Elec_6.3x7.7 -> Capacitor_SMD:C_1206_3216Metric
- C22: renamed from C46; footprint Capacitor_SMD:CP_Elec_6.3x7.7 -> Capacitor_SMD:C_0402_1005Metric
- C26: renamed from C63; footprint Capacitor_SMD:CP_Elec_6.3x7.7 -> Capacitor_SMD:C_0402_1005Metric
- C27: renamed from C50; footprint Capacitor_SMD:CP_Elec_6.3x7.7 -> Capacitor_SMD:C_0402_1005Metric
- C28: renamed from C57; footprint Capacitor_SMD:CP_Elec_6.3x7.7 -> Capacitor_SMD:C_0402_1005Metric
- C29: renamed from C43; footprint Capacitor_SMD:CP_Elec_6.3x7.7 -> Capacitor_SMD:C_0402_1005Metric
- C32: renamed from C64; footprint Capacitor_SMD:CP_Elec_6.3x7.7 -> Capacitor_SMD:C_0402_1005Metric
- C33: renamed from C51; footprint Capacitor_SMD:CP_Elec_6.3x7.7 -> Capacitor_SMD:C_0402_1005Metric
- C34: renamed from C58; footprint Capacitor_SMD:CP_Elec_6.3x7.7 -> Capacitor_SMD:C_0402_1005Metric
- C36: renamed from C71; footprint Capacitor_SMD:CP_Elec_6.3x7.7 -> Capacitor_SMD:C_0402_1005Metric
- C37: renamed from C73; footprint Capacitor_SMD:CP_Elec_6.3x7.7 -> Capacitor_SMD:C_0402_1005Metric
- C42: renamed from C72; footprint Capacitor_SMD:CP_Elec_6.3x7.7 -> Capacitor_SMD:C_0402_1005Metric
- C43: renamed from C74; footprint Capacitor_SMD:CP_Elec_6.3x7.7 -> Capacitor_SMD:C_0402_1005Metric
- C44: renamed from C66; footprint Capacitor_SMD:CP_Elec_6.3x7.7 -> Capacitor_SMD:C_0402_1005Metric
- C45: renamed from C54; footprint Capacitor_SMD:CP_Elec_6.3x7.7 -> Capacitor_SMD:C_0402_1005Metric
- C46: renamed from C60; footprint Capacitor_SMD:CP_Elec_6.3x7.7 -> Capacitor_SMD:C_0402_1005Metric
- C47: renamed from C75; footprint Capacitor_SMD:CP_Elec_6.3x7.7 -> Capacitor_SMD:C_0402_1005Metric
- C48: renamed from C76; footprint Capacitor_SMD:CP_Elec_6.3x7.7 -> Capacitor_SMD:C_0402_1005Metric
- C49: renamed from C67; footprint Capacitor_SMD:CP_Elec_6.3x7.7 -> Capacitor_SMD:C_0402_1005Metric
- C50: renamed from C55; footprint Capacitor_SMD:CP_Elec_6.3x7.7 -> Capacitor_SMD:C_0402_1005Metric
- C51: renamed from C61; footprint Capacitor_SMD:CP_Elec_6.3x7.7 -> Capacitor_SMD:C_0402_1005Metric
- C75: renamed from C23; footprint Capacitor_SMD:CP_Elec_6.3x7.7 -> Capacitor_SMD:C_0402_1005Metric
- IC3: renamed from IC1; footprint SOIC127P1032X265-28N -> IR2136STRPBF:SOIC127P1032X265-28N
- IC4: renamed from IC2; footprint SOIC127P1032X265-28N -> IR2136STRPBF:SOIC127P1032X265-28N
- IC5: renamed from IC3; footprint SOIC127P1032X265-28N -> IR2136STRPBF:SOIC127P1032X265-28N
- IC6: renamed from IC4; footprint SOIC127P1032X265-28N -> IR2136STRPBF:SOIC127P1032X265-28N
- IC7: renamed from IC6; footprint SOIC127P1032X265-28N -> IR2136STRPBF:SOIC127P1032X265-28N
- IC8: renamed from IC5; footprint SOIC127P1032X265-28N -> IR2136STRPBF:SOIC127P1032X265-28N
- U2: renamed from U1; private KLC_S4.2_VREG_LX -> (none)
- renumbered C69 to C12, C70 to C13, C83 to C14, C89 to C15, C82 to C17, C90 to C18, C78 to C21, C62 to C23, C52 to C24, C56 to C25, C47 to C3, C79 to C30, C68 to C31, C80 to C35, C65 to C38, C53 to C39, C86 to C4, C59 to C40, C81 to C41, C92 to C5, C7 to C52, C8 to C53, C15 to C54, C3 to C55, C5 to C57, C4 to C58, C2 to C59, C77 to C6, C6 to C60, C10 to C61, C9 to C62, C12 to C64, C13 to C65, C14 to C66, C16 to C67, C17 to C68, C49 to C7, C19 to C70, C20 to C71, C21 to C72, C22 to C73, C42 to C74, C24 to C76, C25 to C77, C26 to C78, C27 to C79, C87 to C8, C28 to C80, C41 to C81, C35 to C82, C34 to C83, C40 to C84, C39 to C85, C33 to C86, C38 to C87, C32 to C88, C31 to C89, C93 to C9, C37 to C90, C36 to C91, C30 to C92, C29 to C93, D19 to D1, D9 to D10, D10 to D11, D11 to D12, D12 to D13, D18 to D14, D17 to D15, D15 to D17, D14 to D18, D13 to D19, D1 to D2, D2 to D4, D4 to D5, D5 to D6, D6 to D7, D7 to D8, D8 to D9, IC8 to IC1, IC7 to IC2, J10 to J4, J11 to J5, L2 to L1, L1 to L2, Q13 to Q11, Q14 to Q12, Q11 to Q13, Q15 to Q14, Q12 to Q15, Q30 to Q19, Q4 to Q2, Q29 to Q20, Q28 to Q21, Q27 to Q22, Q26 to Q23, Q25 to Q24, Q19 to Q25, Q20 to Q26, Q21 to Q27, Q22 to Q28, Q23 to Q29, Q2 to Q3, Q36 to Q30, Q35 to Q31, Q24 to Q32, Q34 to Q33, Q33 to Q34, Q32 to Q35, Q31 to Q36, Q5 to Q4, Q7 to Q5, Q8 to Q6, Q3 to Q7, Q9 to Q8, Q6 to Q9, R97 to R1, R7 to R10, R9 to R11, R10 to R12, R11 to R13, R12 to R14, R16 to R15, R17 to R16, R18 to R17, R19 to R18, R20 to R19, R91 to R2, R21 to R20, R28 to R21, R29 to R22, R30 to R23, R4 to R24, R31 to R25, R32 to R26, R33 to R27, R3 to R28, R5 to R29, R92 to R3, R6 to R30, R2 to R31, R22 to R32, R1 to R33, R23 to R34, R24 to R35, R25 to R36, R26 to R37, R27 to R38, R34 to R39, R93 to R4, R35 to R40, R36 to R41, R37 to R42, R38 to R43, R39 to R44, R64 to R45, R65 to R46, R66 to R47, R40 to R48, R41 to R49, R94 to R5, R42 to R50, R67 to R51, R68 to R52, R69 to R53, R43 to R54, R44 to R55, R45 to R56, R70 to R57, R71 to R58, R72 to R59, R96 to R6, R63 to R60, R90 to R61, R89 to R62, R62 to R63, R88 to R64, R61 to R65, R60 to R66, R59 to R67, R58 to R68, R46 to R69, R95 to R7, R47 to R70, R48 to R71, R49 to R72, R50 to R73, R51 to R74, R84 to R75, R83 to R76, R82 to R77, R81 to R78, R98 to R8, R54 to R82, R80 to R83, R53 to R84, R52 to R85, R79 to R86, R78 to R87, R77 to R88, R76 to R89, R8 to R9, R75 to R90, R74 to R91, R73 to R92, R15 to R93, R14 to R94, R13 to R95, TP19 to TP1, TP3 to TP10, TP7 to TP11, TP9 to TP12, TP8 to TP13, TP16 to TP14, TP17 to TP15, TP18 to TP16, TP10 to TP17, TP11 to TP18, TP12 to TP19, TP22 to TP2, TP13 to TP20, TP14 to TP21, TP15 to TP22, TP20 to TP3, TP21 to TP4, TP4 to TP5, TP5 to TP7, TP1 to TP8, TP2 to TP9, U16 to U1, U6 to U10, U9 to U11, U12 to U13, U11 to U14, U10 to U15, U2 to U3, U14 to U6, U15 to U7, U3 to U8, U8 to U9
Connections:
- net GND: now also R45.1, R46.1, R47.1, R51.1, R52.1, R53.1, R57.1, R58.1, R59.1
