File: hardware/esc/esc/esc.kicad_sch (KiCad schematic)
At the start: 291 parts, among them IC1 MP9486AGN-Z, IC2 TLA2528IRTER, IC3 IR2136SPBF, IC4 IR2136SPBF, IC5 IR2136SPBF, IC6 IR2136SPBF, IC7 IR2136SPBF, IC8 IR2136SPBF, J1 USB-C, J2 DEBUG, J3 TEMP-GPIO, J4 GPIO, J5 Conn_01x08_Pin, Q1 NMOS, Q10 NMOS, Q11 NMOS, Q12 NMOS, Q13 NMOS, Q14 NMOS, Q15 NMOS, Q16 NMOS, Q17 NMOS, Q18 NMOS, Q19 NMOS, Q2 NMOS, Q20 NMOS, Q21 NMOS, Q22 NMOS, Q23 NMOS, Q24 NMOS, Q25 NMOS, Q26 NMOS, Q27 NMOS, Q28 NMOS, Q29 NMOS, Q3 NMOS, Q30 NMOS, Q31 NMOS, Q32 NMOS, Q33 NMOS, Q34 NMOS, Q35 NMOS, Q36 NMOS, Q4 NMOS, Q5 NMOS, Q6 NMOS, Q7 NMOS, Q8 NMOS, Q9 NMOS, SW1 SW_Push, SW2 SW_Push, U1 AZ1117CH2-3.3, U10 INA240A2PW, U11 INA240A2PW, U13 INA240A2PW, U14 INA240A2PW, U15 INA240A2PW, U2 RP2354B, U3 INA240A2PW, U4 INA240A2PW, U5 INA240A2PW, U6 TMP110D, U7 TMP110D, U8 INA240A2PW, U9 INA240A2PW, Y1 12MHz

Commit message: codex partial
Connections:
- net BEC_SHDN: now also U2.20 (GPIO20); no longer IC2.6 (AIN7/GPIO7), J3.8 (Pin_8)
- net BEC_SHDN2: now also IC2.6 (AIN7/GPIO7), J3.8 (Pin_8); no longer IC2.5 (AIN6/GPIO6), J3.7 (Pin_7)
- net GND: now also C6.1, U1.2 (GND)
- new net: IC2.5 (AIN6/GPIO6), J3.7 (Pin_7)
Changed lines of the file:
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@@
 	)
 	(junction
+		(at 57.15 38.1)
+		(diameter 0)
+		(color 0 0 0 0)
+	)
+	(junction
 		(at 455.93 167.8316)
 		(diameter 0)
@@
 	(wire
 		(pts
+			(xy 80.01 403.86) (xy 405.13 403.86)
+		)
+		(stroke
+			(width 0)
+			(type default)
+		)
+	)
+	(wire
+		(pts
 			(xy 209.55 187.96) (xy 207.01 187.96)
 		)
@@
 	(wire
 		(pts
+			(xy 535.94 158.75) (xy 533.4 158.75)
+		)
+		(stroke
+			(width 0)
+			(type default)
+		)
+	)
+	(wire
+		(pts
 			(xy 138.43 318.77) (xy 138.43 312.42)
 		)
@@
 	(wire
 		(pts
+			(xy 553.72 139.7) (xy 556.26 139.7)
+		)
+		(stroke
+			(width 0)
+			(type default)
+		)
+	)
+	(wire
+		(pts
 			(xy 283.21 351.79) (xy 271.78 351.79)
 		)
@@
 	(wire
 		(pts
-			(xy 537.21 185.42) (xy 528.32 185.42)
-		)
-		(stroke
-			(width 0)
-			(type default)
-		)
-	)
-	(wire
-		(pts
 			(xy 222.25 78.74) (xy 222.25 107.95)
 		)
@@
 	(wire
 		(pts
+			(xy 147.32 222.25) (xy 154.94 222.25)
+		)
+		(stroke
+			(width 0)
+			(type default)
+		)
+	)
+	(wire
+		(pts
 			(xy 110.49 106.68) (xy 110.49 107.95)
 		)
@@
 	(wire
 		(pts
-			(xy 80.01 403.86) (xy 405.13 403.86)
-		)
-		(stroke
-			(width 0)
-			(type default)
-		)
-	)
-	(wire
-		(pts
 			(xy 256.54 204.47) (xy 256.54 217.17)
 		)
@@
 	(wire
 		(pts
-			(xy 537.21 214.63) (xy 537.21 185.42)
-		)
-		(stroke
-			(width 0)
-			(type default)
-		)
-	)
-	(wire
-		(pts
 			(xy 242.57 186.69) (xy 242.57 133.35)
 		)
@@
 	)
 	(label "BEC_SHDN2"
-		(at 124.46 372.11 0)
+		(at 124.46 375.92 0)
 		(effects
 			(font
@@
 	)
 	(label "BEC_SHDN"
-		(at 129.54 375.92 0)
+		(at 154.94 222.25 0)
 		(effects
 			(font
@@
 	)
 	(symbol
+		(lib_id "power:GND")
+		(at 57.15 38.1 0)
+		(unit 1)
+		(exclude_from_sim no)
+		(in_bom yes)
+		(on_board yes)
+		(dnp no)
+		(fields_autoplaced yes)
+		(property "Reference" "#PWR0120"
+			(at 57.15 44.45 0)
+			(effects
+				(font
+					(size 1.27 1.27)
+				)
+				(hide yes)
+			)
+		)
+		(property "Value" "GND"
+			(at 57.15 43.18 0)
+			(effects
+				(font
+					(size 1.27 1.27)
+				)
+			)
+		)
+		(property "Footprint" ""
+			(at 57.15 38.1 0)
+			(effects
+				(font
+					(size 1.27 1.27)
+				)
+				(hide yes)
+			)
+		)
+		(property "Datasheet" ""
+			(at 57.15 38.1 0)
+			(effects
+				(font
+					(size 1.27 1.27)
+				)
+				(hide yes)
+			)
+		)
+		(property "Description" "Power symbol creates a global label with name \"GND\" , ground"
+			(at 57.15 38.1 0)
+			(effects
+				(font
+					(size 1.27 1.27)
+				)
+				(hide yes)
+			)
+		)
+		(pin "1"
+		)
+		(instances
+			(project "esc"
+				(path "/98640010-11bc-4686-91cc-8acbb55a5e3d"
+					(reference "#PWR0120")
+					(unit 1)
+				)
+			)
+		)
+	)
+	(symbol
 		(lib_id "Device:R_Small")
 		(at 251.46 43.18 270)
@@
 	(symbol
 		(lib_id "power:+3V3")
-		(at 556.26 139.7 0)
+		(at 553.72 139.7 0)
 		(unit 1)
 		(exclude_from_sim no)
@@
 		(fields_autoplaced yes)
 		(property "Reference" "#PWR0136"
-			(at 556.26 143.51 0)
+			(at 553.72 143.51 0)
 			(effects
 				(font
@@
 		)
 		(property "Value" "+3V3"
-			(at 556.26 134.62 0)
+			(at 553.72 134.62 0)
 			(effects
 				(font
@@
 		)
 		(property "Footprint" ""
-			(at 556.26 139.7 0)
+			(at 553.72 139.7 0)
 			(effects
 				(font
@@
 		)
 		(property "Datasheet" ""
-			(at 556.26 139.7 0)
+			(at 553.72 139.7 0)
 			(effects
 				(font
@@
 		)
 		(property "Description" "Power symbol creates a global label with name \"+3V3\""
-			(at 556.26 139.7 0)
+			(at 553.72 139.7 0)
 			(effects
 				(font
@@
 	(symbol
 		(lib_id "power:+3V3")
-		(at 533.4 158.75 0)
+		(at 535.94 158.75 0)
 		(unit 1)
 		(exclude_from_sim no)
@@
 		(fields_autoplaced yes)
 		(property "Reference" "#PWR0128"
-			(at 533.4 162.56 0)
+			(at 535.94 162.56 0)
 			(effects
 				(font
@@
 		)
 		(property "Value" "+3V3"
-			(at 533.4 153.67 0)
+			(at 535.94 153.67 0)
 			(effects
 				(font
@@
 		)
 		(property "Footprint" ""
-			(at 533.4 158.75 0)
+			(at 535.94 158.75 0)
 			(effects
 				(font
@@
 		)
 		(property "Datasheet" ""
-			(at 533.4 158.75 0)
+			(at 535.94 158.75 0)
 			(effects
 				(font
@@
 		)
 		(property "Description" "Power symbol creates a global label with name \"+3V3\""
-			(at 533.4 158.75 0)
+			(at 535.94 158.75 0)
 			(effects
 				(font
