File: hardware/main/rev_b/rf_915.kicad_sch (KiCad schematic)
At the start: 56 parts, among them J40 915MHz_ANT, U40 CC1121RHBR, U41 CC1190RGVR, Y40 32MHz NT2016SA-32M-TEE3017A

Commit message: fix: consolidate portable Rev-B hardware sources
Parts:
- C100, C101, C102, C103, C104, C105, C106, C110, C111, C112, C113, C114, C115, C80, C81, C82, C83, C84, C85, C86, C87, C88, C89, C90, C91, C92, C93, C94, C95, C96, FL40, FL41, J40, L40, L41, L42, L43, L44, L45, L46, L47, L48, L49, R40, R41, R42, R43, R44, R45, R46, R47, R50, R51, U40, U41, Y40: hierarchy_path /1aef5005-7133-4d76-81ba-175878f4fb26/efa0f373-a692-4412-a2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 -> /ec8c7281-c7c4-4b94-8ca3-022eb4ab668a/d728c49e-dd81-451e-8b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
