File: hardware/main/rev_b/rf_915.kicad_sch (KiCad schematic)
At the start: 56 parts, among them J40 915MHz_ANT, U40 CC1121RHBR, U41 CC1190RGVR, Y40 32MHz NT2016SA-32M-TEE3017A

Commit message: build: route and validate rev-b boards
Parts:
- C100, C101, C102, C103, C104, C105, C106, C110, C111, C112, C113, C114, C115, C80, C81, C82, C83, C84, C85, C86, C87, C88, C89, C90, C91, C92, C93, C94, C95, C96, FL40, FL41, J40, L40, L41, L42, L43, L44, L45, L46, L47, L48, L49, R40, R41, R42, R43, R44, R45, R46, R47, R50, R51, U40, U41, Y40: hierarchy_path /1aef5005-7133-4d76-81ba-175878f4fb26/efa0f373-a692-4412-a2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 -> /756fa1ee-c1d1-4641-acbe-e478e0cf7ce2/e93687c9-406c-4661-ae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

Commit message: build: route and validate rev-b boards
Parts:
- C100, C101, C102, C103, C104, C105, C106, C110, C111, C112, C113, C114, C115, C80, C81, C82, C83, C84, C85, C86, C87, C88, C89, C90, C91, C92, C93, C94, C95, C96, FL40, FL41, J40, L40, L41, L42, L43, L44, L45, L46, L47, L48, L49, R40, R41, R42, R43, R44, R45, R46, R47, R50, R51, U40, U41, Y40: hierarchy_path /756fa1ee-c1d1-4641-acbe-e478e0cf7ce2/e93687c9-406c-4661-ae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 -> /bc9e88ab-ec71-446d-863b-0a48e263bdad/34e8e03a-397f-4a1b-b9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

Commit message: build: route and validate rev-b boards
Parts:
- C100, C101, C102, C103, C104, C105, C106, C110, C111, C112, C113, C114, C115, C80, C81, C82, C83, C84, C85, C86, C87, C88, C89, C90, C91, C92, C93, C94, C95, C96, FL40, FL41, J40, L40, L41, L42, L43, L44, L45, L46, L47, L48, L49, R40, R41, R42, R43, R44, R45, R46, R47, R50, R51, U40, U41, Y40: hierarchy_path /bc9e88ab-ec71-446d-863b-0a48e263bdad/34e8e03a-397f-4a1b-b9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 -> /9614676e-b386-466d-a8c4-72c158110f92/ba1385e7-89b7-4484-b6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
