File: hardware/main/rev_b/main_rev_b_final.before_diff_pair_ripup.kicad_pcb (KiCad board)
At the start: 4 copper layers, 130 x 74.5 mm, 168 parts, among them J1 USB-C USB2, J10 SWD, J2 ESC_CAN_POWER, J30 GNSS_UFL, J40 915MHz_ANT, J60 ESC_PWM_1, J61 ESC_PWM_2, J62 ESC_PWM_3, J63 ESC_PWM_4, J64 ESC_PWM_5, J65 ESC_PWM_6, Q30 2N7002, U1 USBLC6-2SC6, U10 RP2354B, U2 TLV62569DBVR, U20 ICM-42688-P, U21 LSM6DSO32TR, U22 LPS22DFTR, U3 TLV75528PDBVR, U30 LG77LICMD, U4 TLV75533PDBVR, U40 CC1121RHBR, U41 CC1190RGVR, U50 TCAN3413DR, U51 MCP2518FD-H/QBB, Y1 12MHz ABM8-272-T3, Y40 32MHz NT2016SA-32M-TEE3017A, Y50 40MHz ABM8G

Commit message: esc: replicate hand-routed power copper and free main diff pairs
Routing:
- net /USB_DP: track 0.00 -> 49.4 mm, vias 0 -> 2
- net /USB_DM: track 0.00 -> 33.7 mm, vias 0 -> 2
- net /CANL: track 0.00 -> 23.5 mm
- net /CAN interface/U50_CANH: track 0.00 -> 19.1 mm
- net /CANH: track 0.00 -> 16.0 mm
- net /CAN interface/U50_CANL: track 0.00 -> 10.2 mm
