File: hardware/main/rev_b/main_rev_b_final.kicad_pcb (KiCad board)
At the start: 4 copper layers, 130 x 74.5 mm, 168 parts, among them J1 USB-C USB2, J10 SWD, J2 ESC_CAN_POWER, J30 GNSS_UFL, J40 915MHz_ANT, J60 ESC_PWM_1, J61 ESC_PWM_2, J62 ESC_PWM_3, J63 ESC_PWM_4, J64 ESC_PWM_5, J65 ESC_PWM_6, Q30 2N7002, U1 USBLC6-2SC6, U10 RP2354B, U2 TLV62569DBVR, U20 ICM-42688-P, U21 LSM6DSO32TR, U22 LPS22DFTR, U3 TLV75528PDBVR, U30 LG77LICMD, U4 TLV75533PDBVR, U40 CC1121RHBR, U41 CC1190RGVR, U50 TCAN3413DR, U51 MCP2518FD-H/QBB, Y1 12MHz ABM8-272-T3, Y40 32MHz NT2016SA-32M-TEE3017A, Y50 40MHz ABM8G

Commit message: Route main board CANH transceiver leg
Routing:
- net /CAN interface/U50_CANH: track 0.00 -> 7.68 mm
Changed lines of the file:
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@@
+	)
+	(segment
+		(start 19 17.2)
+		(end 19 19.825)
+		(width 0.2)
+		(layer "F.Cu")
+		(net 41)
+	)
+	(segment
+		(start 19 19.825)
+		(end 20.08 19.825)
+		(width 0.2)
+		(layer "F.Cu")
+		(net 41)
+	)
+	(segment
+		(start 22.105 15.135)
+		(end 21 15.135)
+		(width 0.2)
+		(layer "F.Cu")
+		(net 41)
+	)
+	(segment
+		(start 21 15.135)
+		(end 19 17.2)
+		(width 0.2)
+		(layer "F.Cu")
+		(net 41)
 	)
 	(segment

Commit message: revert ESC to front-side-only placement from 325f93b; main board CANL routing + ACT45B pinout fix
Routing:
- net /CAN interface/U50_CANL: track 0.00 -> 6.77 mm, vias 0 -> 2
Changed lines of the file:
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@@
+	)
+	(segment
+		(start 22.105 13.865)
+		(end 20 13.865)
+		(width 0.2)
+		(layer "F.Cu")
+		(net 42)
+	)
+	(segment
+		(start 20.8 17.3)
+		(end 20.08 18.175)
+		(width 0.2)
+		(layer "F.Cu")
+		(net 42)
+	)
+	(via
+		(at 20 13.865)
+		(size 0.6)
+		(drill 0.3)
+		(layers "F.Cu" "B.Cu")
+		(net 42)
+	)
+	(via
+		(at 20.8 17.3)
+		(size 0.6)
+		(drill 0.3)
+		(layers "F.Cu" "B.Cu")
+		(net 42)
+	)
+	(segment
+		(start 20 13.865)
+		(end 20.8 17.3)
+		(width 0.2)
+		(layer "B.Cu")
+		(net 42)
 	)
 	(segment
