File: hardware/main/rev_b/main_rev_b.kicad_pcb (KiCad board)
At the start: 4 copper layers, 140 x 100 mm, 165 parts, among them J1 USB-C USB2, J10 SWD, J2 ESC_CAN_POWER, J30 GNSS_UFL, J40 915MHz_ANT, Q30 2N7002, U1 USBLC6-2SC6, U10 RP2354B, U2 TLV62569DBVR, U20 ICM-42688-P, U21 LSM6DSO32TR, U22 LPS22DFTR, U3 TLV75528PDBVR, U30 LG77LICMD, U4 TLV75533PDBVR, U40 CC1121RHBR, U41 CC1190RGVR, U50 TCAN3413DR, U51 MCP2518FD-H/QBB, Y1 12MHz ABM8-272-T3, Y40 32MHz NT2016SA-32M-TEE3017A, Y50 40MHz ABM8G

Commit message: pcb: connect local rev b 3v3 islands
Routing:
- net /3V3: track 19.2 -> 24.5 mm
Changed lines of the file:
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@@
+	)
+	(segment
+		(start 59.52 43.5)
+		(end 58.8 42.78)
+		(width 0.2)
+		(layer "F.Cu")
+		(net 3)
 	)
 	(segment
@@
 	)
 	(segment
+		(start 58.8 42.78)
+		(end 61.6 42.78)
+		(width 0.2)
+		(layer "F.Cu")
+		(net 3)
+	)
+	(segment
 		(start 62.52 44.3)
 		(end 62.52 43.5)
@@
 		(width 0.2)
 		(layer "F.Cu")
+		(net 3)
+	)
+	(segment
+		(start 61.6 42.78)
+		(end 61.6 44.3)
+		(width 0.2)
+		(layer "F.Cu")

Commit message: pcb: route second local rev b 3v3 island
Routing:
- net /3V3: track 24.5 -> 31.4 mm
Changed lines of the file:
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@@
+	)
+	(segment
+		(start 64.7 42.5)
+		(end 64.7 46.2)
+		(width 0.2)
+		(layer "F.Cu")
+		(net 3)
 	)
 	(segment
@@
 		(width 0.2)
 		(layer "F.Cu")
+		(net 3)
+	)
+	(segment
+		(start 62.52 42.5)
+		(end 64.7 42.5)
+		(width 0.2)
+		(layer "F.Cu")
+		(net 3)
+	)
+	(segment
+		(start 62.52 43.5)
+		(end 62.52 42.5)
+		(width 0.2)
+		(layer "F.Cu")

Commit message: pcb: route northwest rev b 3v3 link
Routing:
- net /3V3: track 31.4 -> 35.6 mm
Changed lines of the file:
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@@
+	)
+	(segment
+		(start 58.8 42.2)
+		(end 56.52 42.2)
+		(width 0.2)
+		(layer "F.Cu")
+		(net 3)
 	)
 	(segment
@@
 	)
 	(segment
+		(start 56.52 42.2)
+		(end 56.52 43.5)
+		(width 0.2)
+		(layer "F.Cu")
+		(net 3)
+	)
+	(segment
 		(start 54.05 51.8)
 		(end 53.4 51.8)
@@
 		(width 0.2)
 		(layer "F.Cu")
+		(net 3)
+	)
+	(segment
+		(start 58.8 42.78)
+		(end 58.8 42.2)
+		(width 0.2)
+		(layer "F.Cu")

Commit message: pcb: connect rev b mcu 3v3 branch
Routing:
- net /3V3: track 35.6 -> 43.4 mm
Changed lines of the file:
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@@
+	)
+	(segment
+		(start 54.05 47.8)
+		(end 53.3 47.8)
+		(width 0.2)
+		(layer "F.Cu")
+		(net 3)
 	)
 	(segment
@@
 		(width 0.2)
 		(layer "F.Cu")
+		(net 3)
+	)
+	(segment
+		(start 53.3 44.2)
+		(end 56.8 44.2)
+		(width 0.2)
+		(layer "F.Cu")
+		(net 3)
+	)
+	(segment
+		(start 53.3 47.8)
+		(end 53.3 44.2)
+		(width 0.2)
+		(layer "F.Cu")

Commit message: pcb: route southwest rev b 3v3 branch
Routing:
- net /3V3: track 43.4 -> 51.9 mm
Changed lines of the file:
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@@
+	)
+	(segment
+		(start 56.4 54.95)
+		(end 56.4 55.7)
+		(width 0.2)
+		(layer "F.Cu")
+		(net 3)
+	)
+	(segment
+		(start 53.3 55.7)
+		(end 53.3 51.8)
+		(width 0.2)
+		(layer "F.Cu")
+		(net 3)
+	)
+	(segment
+		(start 53.3 51.8)
+		(end 54.05 51.8)
+		(width 0.2)
+		(layer "F.Cu")
+		(net 3)
 	)
 	(segment
@@
 		(width 0.2)
 		(layer "F.Cu")
+		(net 3)
+	)
+	(segment
+		(start 56.4 55.7)
+		(end 53.3 55.7)
+		(width 0.2)
+		(layer "F.Cu")

Commit message: pcb: add south edge rev b 3v3 route
Routing:
- net /3V3: track 51.9 -> 54.7 mm
Changed lines of the file:
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@@
+	)
+	(segment
+		(start 58.4 54.95)
+		(end 58.4 55.7)
+		(width 0.2)
+		(layer "F.Cu")
+		(net 3)
 	)
 	(segment
@@
 		(width 0.2)
 		(layer "F.Cu")
+		(net 3)
+	)
+	(segment
+		(start 58.4 55.7)
+		(end 56.4 55.7)
+		(width 0.2)
+		(layer "F.Cu")
