File: hardware/esc/rev_b/quilter_upload/motor_1.kicad_sch (KiCad schematic)
At the start: 94 parts, among them J1101 FUSED_BATTERY_TAP, J1102 MOTOR_PHASES, J1103 LOCAL_SWD, Q1101 IPTC014N10NM5, Q1102 IPTC014N10NM5, Q1103 IPTC014N10NM5, Q1104 IPTC014N10NM5, Q1105 IPTC014N10NM5, Q1106 IPTC014N10NM5, U1101 DRV8353SRTAR, U1102 STM32G431CBT6, U1103 ISO6731FDWR, U1104 TPS70933DBVR, U1105 INA296A2IDR, U1106 SN74LVC1G08DBVR, Y1101 8MHz ABM8G

Commit message: Package ESC USB design for Quilter
Parts:
- removed C1130: 820u 100V, Capacitor_THT:CP_Radial_D18.0mm_P7.50mm, symbol Device:C_Polarized
- added J1104: USB_DFU_SERVICE, Connector_JST:JST_GH_SM06B-GHS-TB_1x06-1MP_P1.25mm_Horizontal, symbol Connector_Generic:Conn_01x06
- added R1180: 100k, Resistor_SMD:R_0603_1608Metric, symbol Device:R
- added R1181: 47k, Resistor_SMD:R_0603_1608Metric, symbol Device:R
- added R1182, R1183, R1184: 0, Resistor_SMD:R_0603_1608Metric, symbol Device:R
- added U1107: USBLC6-2SC6, Package_TO_SOT_SMD:SOT-23-6, symbol revb:USBLC6-2SC6
- C1101, C1102, C1103, C1104, C1105, C1106, C1107, C1120, C1121, C1122, C1123, C1131, C1132, C1133, C1134, C1135, C1136, C1150, C1160, C1161, C1162, C1163, C1164, C1165, C1166, C1167, C1168, C1169, C1170, C1171, C1172, C1173, C1174, C1175, C1176, C1177, D1101, D1102, FB1101, J1101, J1102, J1103, PS1101, Q1101, Q1102, Q1103, Q1104, Q1105, Q1106, R1101, R1102, R1103, R1104, R1105, R1106, R1107, R1108, R1109, R1110, R1111, R1112, R1120, R1121, R1122, R1123, R1130, R1131, R1132, R1133, R1140, R1141, R1142, R1143, R1144, R1145, R1150, R1151, R1152, R1153, R1154, R1155, R1156, R1157, R1158, R1159, TH1, U1101, U1102, U1103, U1104, U1105, U1106, Y1101: hierarchy_path /98734485-5dd9-43e3-8e43-27cf828371fb/f46d8a37-3270-48b3-ad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 -> /9645d861-d8e4-412a-9066-8076bbd6b1f6/6f4ffbb4-5135-4088-8b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
Connections:
- net M1_ARM_ISO: now also U1102.25 (PB11); no longer U1102.34 (PA12)
- net M1_BATN: now also R1181.2, R1182.2, U1107.2 (GND)
- net M1_BOOT0: now also R1183.2
- net M1_DRV_nFAULT: now also U1102.22 (PB10); no longer U1102.33 (PA11)
- net M1_NRST: now also R1184.2
- new net M1_USB_BOOT0: J1104.5 (Pin_5), R1183.1
- new net M1_USB_DM: J1104.2 (Pin_2), U1102.33 (PA11), U1107.1 (IO1), U1107.6 (IO1)
- new net M1_USB_DP: J1104.1 (Pin_1), U1102.34 (PA12), U1107.3 (IO2), U1107.4 (IO2)
- new net M1_USB_GND: J1104.3 (Pin_3), R1182.1
- new net M1_USB_NRST: J1104.6 (Pin_6), R1184.1
- new net M1_USB_VBUS: J1104.4 (Pin_4), R1180.1, U1107.5 (VBUS)
- new net M1_USB_VBUS_SENSE: R1180.2, R1181.1
- no-connect marks 13 -> 11
Other:
- note added: "C1130 is external: connect bulk capacitance directly across M1_BATP/M1_BATN with the shortest practical high-current loop."
