File: hardware/esc/rev_b/quilter_upload/motor_2.kicad_sch (KiCad schematic)
At the start: 94 parts, among them J1201 FUSED_BATTERY_TAP, J1202 MOTOR_PHASES, J1203 LOCAL_SWD, Q1201 IPTC014N10NM5, Q1202 IPTC014N10NM5, Q1203 IPTC014N10NM5, Q1204 IPTC014N10NM5, Q1205 IPTC014N10NM5, Q1206 IPTC014N10NM5, U1201 DRV8353SRTAR, U1202 STM32G431CBT6, U1203 ISO6731FDWR, U1204 TPS70933DBVR, U1205 INA296A2IDR, U1206 SN74LVC1G08DBVR, Y1201 8MHz ABM8G

Commit message: Package ESC USB design for Quilter
Parts:
- removed C1230: 820u 100V, Capacitor_THT:CP_Radial_D18.0mm_P7.50mm, symbol Device:C_Polarized
- added J1204: USB_DFU_SERVICE, Connector_JST:JST_GH_SM06B-GHS-TB_1x06-1MP_P1.25mm_Horizontal, symbol Connector_Generic:Conn_01x06
- added R1280: 100k, Resistor_SMD:R_0603_1608Metric, symbol Device:R
- added R1281: 47k, Resistor_SMD:R_0603_1608Metric, symbol Device:R
- added R1282, R1283, R1284: 0, Resistor_SMD:R_0603_1608Metric, symbol Device:R
- added U1207: USBLC6-2SC6, Package_TO_SOT_SMD:SOT-23-6, symbol revb:USBLC6-2SC6
- C1201, C1202, C1203, C1204, C1205, C1206, C1207, C1220, C1221, C1222, C1223, C1231, C1232, C1233, C1234, C1235, C1236, C1250, C1260, C1261, C1262, C1263, C1264, C1265, C1266, C1267, C1268, C1269, C1270, C1271, C1272, C1273, C1274, C1275, C1276, C1277, D1201, D1202, FB1201, J1201, J1202, J1203, PS1201, Q1201, Q1202, Q1203, Q1204, Q1205, Q1206, R1201, R1202, R1203, R1204, R1205, R1206, R1207, R1208, R1209, R1210, R1211, R1212, R1220, R1221, R1222, R1223, R1230, R1231, R1232, R1233, R1240, R1241, R1242, R1243, R1244, R1245, R1250, R1251, R1252, R1253, R1254, R1255, R1256, R1257, R1258, R1259, TH2, U1201, U1202, U1203, U1204, U1205, U1206, Y1201: hierarchy_path /98734485-5dd9-43e3-8e43-27cf828371fb/356e025b-7dfd-46c7-b8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 -> /9645d861-d8e4-412a-9066-8076bbd6b1f6/d850c5a2-6df1-4c7e-b7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
Connections:
- net M2_ARM_ISO: now also U1202.25 (PB11); no longer U1202.34 (PA12)
- net M2_BATN: now also R1281.2, R1282.2, U1207.2 (GND)
- net M2_BOOT0: now also R1283.2
- net M2_DRV_nFAULT: now also U1202.22 (PB10); no longer U1202.33 (PA11)
- net M2_NRST: now also R1284.2
- new net M2_USB_BOOT0: J1204.5 (Pin_5), R1283.1
- new net M2_USB_DM: J1204.2 (Pin_2), U1202.33 (PA11), U1207.1 (IO1), U1207.6 (IO1)
- new net M2_USB_DP: J1204.1 (Pin_1), U1202.34 (PA12), U1207.3 (IO2), U1207.4 (IO2)
- new net M2_USB_GND: J1204.3 (Pin_3), R1282.1
- new net M2_USB_NRST: J1204.6 (Pin_6), R1284.1
- new net M2_USB_VBUS: J1204.4 (Pin_4), R1280.1, U1207.5 (VBUS)
- new net M2_USB_VBUS_SENSE: R1280.2, R1281.1
- no-connect marks 13 -> 11
Other:
- note added: "C1230 is external: connect bulk capacitance directly across M2_BATP/M2_BATN with the shortest practical high-current loop."
