File: hardware/esc/rev_b/quilter_upload/motor_3.kicad_sch (KiCad schematic)
At the start: 94 parts, among them J1301 FUSED_BATTERY_TAP, J1302 MOTOR_PHASES, J1303 LOCAL_SWD, Q1301 IPTC014N10NM5, Q1302 IPTC014N10NM5, Q1303 IPTC014N10NM5, Q1304 IPTC014N10NM5, Q1305 IPTC014N10NM5, Q1306 IPTC014N10NM5, U1301 DRV8353SRTAR, U1302 STM32G431CBT6, U1303 ISO6731FDWR, U1304 TPS70933DBVR, U1305 INA296A2IDR, U1306 SN74LVC1G08DBVR, Y1301 8MHz ABM8G

Commit message: Package ESC USB design for Quilter
Parts:
- removed C1330: 820u 100V, Capacitor_THT:CP_Radial_D18.0mm_P7.50mm, symbol Device:C_Polarized
- added J1304: USB_DFU_SERVICE, Connector_JST:JST_GH_SM06B-GHS-TB_1x06-1MP_P1.25mm_Horizontal, symbol Connector_Generic:Conn_01x06
- added R1380: 100k, Resistor_SMD:R_0603_1608Metric, symbol Device:R
- added R1381: 47k, Resistor_SMD:R_0603_1608Metric, symbol Device:R
- added R1382, R1383, R1384: 0, Resistor_SMD:R_0603_1608Metric, symbol Device:R
- added U1307: USBLC6-2SC6, Package_TO_SOT_SMD:SOT-23-6, symbol revb:USBLC6-2SC6
- C1301, C1302, C1303, C1304, C1305, C1306, C1307, C1320, C1321, C1322, C1323, C1331, C1332, C1333, C1334, C1335, C1336, C1350, C1360, C1361, C1362, C1363, C1364, C1365, C1366, C1367, C1368, C1369, C1370, C1371, C1372, C1373, C1374, C1375, C1376, C1377, D1301, D1302, FB1301, J1301, J1302, J1303, PS1301, Q1301, Q1302, Q1303, Q1304, Q1305, Q1306, R1301, R1302, R1303, R1304, R1305, R1306, R1307, R1308, R1309, R1310, R1311, R1312, R1320, R1321, R1322, R1323, R1330, R1331, R1332, R1333, R1340, R1341, R1342, R1343, R1344, R1345, R1350, R1351, R1352, R1353, R1354, R1355, R1356, R1357, R1358, R1359, TH3, U1301, U1302, U1303, U1304, U1305, U1306, Y1301: hierarchy_path /98734485-5dd9-43e3-8e43-27cf828371fb/da8728a6-f28b-47de-93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 -> /9645d861-d8e4-412a-9066-8076bbd6b1f6/2646df52-a79d-4dd5-9a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
Connections:
- net M3_ARM_ISO: now also U1302.25 (PB11); no longer U1302.34 (PA12)
- net M3_BATN: now also R1381.2, R1382.2, U1307.2 (GND)
- net M3_BOOT0: now also R1383.2
- net M3_DRV_nFAULT: now also U1302.22 (PB10); no longer U1302.33 (PA11)
- net M3_NRST: now also R1384.2
- new net M3_USB_BOOT0: J1304.5 (Pin_5), R1383.1
- new net M3_USB_DM: J1304.2 (Pin_2), U1302.33 (PA11), U1307.1 (IO1), U1307.6 (IO1)
- new net M3_USB_DP: J1304.1 (Pin_1), U1302.34 (PA12), U1307.3 (IO2), U1307.4 (IO2)
- new net M3_USB_GND: J1304.3 (Pin_3), R1382.1
- new net M3_USB_NRST: J1304.6 (Pin_6), R1384.1
- new net M3_USB_VBUS: J1304.4 (Pin_4), R1380.1, U1307.5 (VBUS)
- new net M3_USB_VBUS_SENSE: R1380.2, R1381.1
- no-connect marks 13 -> 11
Other:
- note added: "C1330 is external: connect bulk capacitance directly across M3_BATP/M3_BATN with the shortest practical high-current loop."
