File: hardware/esc/rev_b/quilter_upload/motor_4.kicad_sch (KiCad schematic)
At the start: 94 parts, among them J1401 FUSED_BATTERY_TAP, J1402 MOTOR_PHASES, J1403 LOCAL_SWD, Q1401 IPTC014N10NM5, Q1402 IPTC014N10NM5, Q1403 IPTC014N10NM5, Q1404 IPTC014N10NM5, Q1405 IPTC014N10NM5, Q1406 IPTC014N10NM5, U1401 DRV8353SRTAR, U1402 STM32G431CBT6, U1403 ISO6731FDWR, U1404 TPS70933DBVR, U1405 INA296A2IDR, U1406 SN74LVC1G08DBVR, Y1401 8MHz ABM8G

Commit message: Package ESC USB design for Quilter
Parts:
- removed C1430: 820u 100V, Capacitor_THT:CP_Radial_D18.0mm_P7.50mm, symbol Device:C_Polarized
- added J1404: USB_DFU_SERVICE, Connector_JST:JST_GH_SM06B-GHS-TB_1x06-1MP_P1.25mm_Horizontal, symbol Connector_Generic:Conn_01x06
- added R1480: 100k, Resistor_SMD:R_0603_1608Metric, symbol Device:R
- added R1481: 47k, Resistor_SMD:R_0603_1608Metric, symbol Device:R
- added R1482, R1483, R1484: 0, Resistor_SMD:R_0603_1608Metric, symbol Device:R
- added U1407: USBLC6-2SC6, Package_TO_SOT_SMD:SOT-23-6, symbol revb:USBLC6-2SC6
- C1401, C1402, C1403, C1404, C1405, C1406, C1407, C1420, C1421, C1422, C1423, C1431, C1432, C1433, C1434, C1435, C1436, C1450, C1460, C1461, C1462, C1463, C1464, C1465, C1466, C1467, C1468, C1469, C1470, C1471, C1472, C1473, C1474, C1475, C1476, C1477, D1401, D1402, FB1401, J1401, J1402, J1403, PS1401, Q1401, Q1402, Q1403, Q1404, Q1405, Q1406, R1401, R1402, R1403, R1404, R1405, R1406, R1407, R1408, R1409, R1410, R1411, R1412, R1420, R1421, R1422, R1423, R1430, R1431, R1432, R1433, R1440, R1441, R1442, R1443, R1444, R1445, R1450, R1451, R1452, R1453, R1454, R1455, R1456, R1457, R1458, R1459, TH4, U1401, U1402, U1403, U1404, U1405, U1406, Y1401: hierarchy_path /98734485-5dd9-43e3-8e43-27cf828371fb/b9f555c6-2b25-4489-8e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 -> /9645d861-d8e4-412a-9066-8076bbd6b1f6/468fe66e-d6f5-40b9-aa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
Connections:
- net M4_ARM_ISO: now also U1402.25 (PB11); no longer U1402.34 (PA12)
- net M4_BATN: now also R1481.2, R1482.2, U1407.2 (GND)
- net M4_BOOT0: now also R1483.2
- net M4_DRV_nFAULT: now also U1402.22 (PB10); no longer U1402.33 (PA11)
- net M4_NRST: now also R1484.2
- new net M4_USB_BOOT0: J1404.5 (Pin_5), R1483.1
- new net M4_USB_DM: J1404.2 (Pin_2), U1402.33 (PA11), U1407.1 (IO1), U1407.6 (IO1)
- new net M4_USB_DP: J1404.1 (Pin_1), U1402.34 (PA12), U1407.3 (IO2), U1407.4 (IO2)
- new net M4_USB_GND: J1404.3 (Pin_3), R1482.1
- new net M4_USB_NRST: J1404.6 (Pin_6), R1484.1
- new net M4_USB_VBUS: J1404.4 (Pin_4), R1480.1, U1407.5 (VBUS)
- new net M4_USB_VBUS_SENSE: R1480.2, R1481.1
- no-connect marks 13 -> 11
Other:
- note added: "C1430 is external: connect bulk capacitance directly across M4_BATP/M4_BATN with the shortest practical high-current loop."
