File: hardware/esc/rev_b/quilter_upload/motor_5.kicad_sch (KiCad schematic)
At the start: 94 parts, among them J1501 FUSED_BATTERY_TAP, J1502 MOTOR_PHASES, J1503 LOCAL_SWD, Q1501 IPTC014N10NM5, Q1502 IPTC014N10NM5, Q1503 IPTC014N10NM5, Q1504 IPTC014N10NM5, Q1505 IPTC014N10NM5, Q1506 IPTC014N10NM5, U1501 DRV8353SRTAR, U1502 STM32G431CBT6, U1503 ISO6731FDWR, U1504 TPS70933DBVR, U1505 INA296A2IDR, U1506 SN74LVC1G08DBVR, Y1501 8MHz ABM8G

Commit message: Package ESC USB design for Quilter
Parts:
- removed C1530: 820u 100V, Capacitor_THT:CP_Radial_D18.0mm_P7.50mm, symbol Device:C_Polarized
- added J1504: USB_DFU_SERVICE, Connector_JST:JST_GH_SM06B-GHS-TB_1x06-1MP_P1.25mm_Horizontal, symbol Connector_Generic:Conn_01x06
- added R1580: 100k, Resistor_SMD:R_0603_1608Metric, symbol Device:R
- added R1581: 47k, Resistor_SMD:R_0603_1608Metric, symbol Device:R
- added R1582, R1583, R1584: 0, Resistor_SMD:R_0603_1608Metric, symbol Device:R
- added U1507: USBLC6-2SC6, Package_TO_SOT_SMD:SOT-23-6, symbol revb:USBLC6-2SC6
- C1501, C1502, C1503, C1504, C1505, C1506, C1507, C1520, C1521, C1522, C1523, C1531, C1532, C1533, C1534, C1535, C1536, C1550, C1560, C1561, C1562, C1563, C1564, C1565, C1566, C1567, C1568, C1569, C1570, C1571, C1572, C1573, C1574, C1575, C1576, C1577, D1501, D1502, FB1501, J1501, J1502, J1503, PS1501, Q1501, Q1502, Q1503, Q1504, Q1505, Q1506, R1501, R1502, R1503, R1504, R1505, R1506, R1507, R1508, R1509, R1510, R1511, R1512, R1520, R1521, R1522, R1523, R1530, R1531, R1532, R1533, R1540, R1541, R1542, R1543, R1544, R1545, R1550, R1551, R1552, R1553, R1554, R1555, R1556, R1557, R1558, R1559, TH5, U1501, U1502, U1503, U1504, U1505, U1506, Y1501: hierarchy_path /98734485-5dd9-43e3-8e43-27cf828371fb/2168df58-a755-415a-91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 -> /9645d861-d8e4-412a-9066-8076bbd6b1f6/0a8863de-3628-49a5-bb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
Connections:
- net M5_ARM_ISO: now also U1502.25 (PB11); no longer U1502.34 (PA12)
- net M5_BATN: now also R1581.2, R1582.2, U1507.2 (GND)
- net M5_BOOT0: now also R1583.2
- net M5_DRV_nFAULT: now also U1502.22 (PB10); no longer U1502.33 (PA11)
- net M5_NRST: now also R1584.2
- new net M5_USB_BOOT0: J1504.5 (Pin_5), R1583.1
- new net M5_USB_DM: J1504.2 (Pin_2), U1502.33 (PA11), U1507.1 (IO1), U1507.6 (IO1)
- new net M5_USB_DP: J1504.1 (Pin_1), U1502.34 (PA12), U1507.3 (IO2), U1507.4 (IO2)
- new net M5_USB_GND: J1504.3 (Pin_3), R1582.1
- new net M5_USB_NRST: J1504.6 (Pin_6), R1584.1
- new net M5_USB_VBUS: J1504.4 (Pin_4), R1580.1, U1507.5 (VBUS)
- new net M5_USB_VBUS_SENSE: R1580.2, R1581.1
- no-connect marks 13 -> 11
Other:
- note added: "C1530 is external: connect bulk capacitance directly across M5_BATP/M5_BATN with the shortest practical high-current loop."
