File: hardware/esc/rev_b/quilter_upload/motor_6.kicad_sch (KiCad schematic)
At the start: 94 parts, among them J1601 FUSED_BATTERY_TAP, J1602 MOTOR_PHASES, J1603 LOCAL_SWD, Q1601 IPTC014N10NM5, Q1602 IPTC014N10NM5, Q1603 IPTC014N10NM5, Q1604 IPTC014N10NM5, Q1605 IPTC014N10NM5, Q1606 IPTC014N10NM5, U1601 DRV8353SRTAR, U1602 STM32G431CBT6, U1603 ISO6731FDWR, U1604 TPS70933DBVR, U1605 INA296A2IDR, U1606 SN74LVC1G08DBVR, Y1601 8MHz ABM8G

Commit message: Package ESC USB design for Quilter
Parts:
- removed C1630: 820u 100V, Capacitor_THT:CP_Radial_D18.0mm_P7.50mm, symbol Device:C_Polarized
- added J1604: USB_DFU_SERVICE, Connector_JST:JST_GH_SM06B-GHS-TB_1x06-1MP_P1.25mm_Horizontal, symbol Connector_Generic:Conn_01x06
- added R1680: 100k, Resistor_SMD:R_0603_1608Metric, symbol Device:R
- added R1681: 47k, Resistor_SMD:R_0603_1608Metric, symbol Device:R
- added R1682, R1683, R1684: 0, Resistor_SMD:R_0603_1608Metric, symbol Device:R
- added U1607: USBLC6-2SC6, Package_TO_SOT_SMD:SOT-23-6, symbol revb:USBLC6-2SC6
- C1601, C1602, C1603, C1604, C1605, C1606, C1607, C1620, C1621, C1622, C1623, C1631, C1632, C1633, C1634, C1635, C1636, C1650, C1660, C1661, C1662, C1663, C1664, C1665, C1666, C1667, C1668, C1669, C1670, C1671, C1672, C1673, C1674, C1675, C1676, C1677, D1601, D1602, FB1601, J1601, J1602, J1603, PS1601, Q1601, Q1602, Q1603, Q1604, Q1605, Q1606, R1601, R1602, R1603, R1604, R1605, R1606, R1607, R1608, R1609, R1610, R1611, R1612, R1620, R1621, R1622, R1623, R1630, R1631, R1632, R1633, R1640, R1641, R1642, R1643, R1644, R1645, R1650, R1651, R1652, R1653, R1654, R1655, R1656, R1657, R1658, R1659, TH6, U1601, U1602, U1603, U1604, U1605, U1606, Y1601: hierarchy_path /98734485-5dd9-43e3-8e43-27cf828371fb/b2d39697-c105-489c-82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 -> /9645d861-d8e4-412a-9066-8076bbd6b1f6/1d5f9359-dc7b-47d9-a6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
Connections:
- net M6_ARM_ISO: now also U1602.25 (PB11); no longer U1602.34 (PA12)
- net M6_BATN: now also R1681.2, R1682.2, U1607.2 (GND)
- net M6_BOOT0: now also R1683.2
- net M6_DRV_nFAULT: now also U1602.22 (PB10); no longer U1602.33 (PA11)
- net M6_NRST: now also R1684.2
- new net M6_USB_BOOT0: J1604.5 (Pin_5), R1683.1
- new net M6_USB_DM: J1604.2 (Pin_2), U1602.33 (PA11), U1607.1 (IO1), U1607.6 (IO1)
- new net M6_USB_DP: J1604.1 (Pin_1), U1602.34 (PA12), U1607.3 (IO2), U1607.4 (IO2)
- new net M6_USB_GND: J1604.3 (Pin_3), R1682.1
- new net M6_USB_NRST: J1604.6 (Pin_6), R1684.1
- new net M6_USB_VBUS: J1604.4 (Pin_4), R1680.1, U1607.5 (VBUS)
- new net M6_USB_VBUS_SENSE: R1680.2, R1681.1
- no-connect marks 13 -> 11
Other:
- note added: "C1630 is external: connect bulk capacitance directly across M6_BATP/M6_BATN with the shortest practical high-current loop."
