File: hardware/esc/rev_b/quilter_upload/esc_rev_b.kicad_pcb (KiCad board)
At the start: 6 copper layers, 150 x 150 mm, 646 parts, among them J1101 FUSED_BATTERY_TAP, J1102 MOTOR_PHASES, J1103 LOCAL_SWD, J1201 FUSED_BATTERY_TAP, J1202 MOTOR_PHASES, J1203 LOCAL_SWD, J1301 FUSED_BATTERY_TAP, J1302 MOTOR_PHASES, J1303 LOCAL_SWD, J1401 FUSED_BATTERY_TAP, J1402 MOTOR_PHASES, J1403 LOCAL_SWD, J1501 FUSED_BATTERY_TAP, J1502 MOTOR_PHASES, J1503 LOCAL_SWD, J1601 FUSED_BATTERY_TAP, J1602 MOTOR_PHASES, J1603 LOCAL_SWD, J201 ESC_SWD, J701 AUX_BATTERY, J702 FLIGHT_CAN_POWER, Q1101 IPTC014N10NM5, Q1102 IPTC014N10NM5, Q1103 IPTC014N10NM5, Q1104 IPTC014N10NM5, Q1105 IPTC014N10NM5, Q1106 IPTC014N10NM5, Q1201 IPTC014N10NM5, Q1202 IPTC014N10NM5, Q1203 IPTC014N10NM5, Q1204 IPTC014N10NM5, Q1205 IPTC014N10NM5, Q1206 IPTC014N10NM5, Q1301 IPTC014N10NM5, Q1302 IPTC014N10NM5, Q1303 IPTC014N10NM5, Q1304 IPTC014N10NM5, Q1305 IPTC014N10NM5, Q1306 IPTC014N10NM5, Q1401 IPTC014N10NM5, Q1402 IPTC014N10NM5, Q1403 IPTC014N10NM5, Q1404 IPTC014N10NM5, Q1405 IPTC014N10NM5, Q1406 IPTC014N10NM5, Q1501 IPTC014N10NM5, Q1502 IPTC014N10NM5, Q1503 IPTC014N10NM5, Q1504 IPTC014N10NM5, Q1505 IPTC014N10NM5, Q1506 IPTC014N10NM5, Q1601 IPTC014N10NM5, Q1602 IPTC014N10NM5, Q1603 IPTC014N10NM5, Q1604 IPTC014N10NM5, Q1605 IPTC014N10NM5, Q1606 IPTC014N10NM5, U1101 DRV8353SRTAR, U1102 STM32G431CBT6, U1103 ISO6731FDWR, U1104 TPS70933DBVR, U1105 INA296A2IDR, U1106 SN74LVC1G08DBVR, U1201 DRV8353SRTAR, U1202 STM32G431CBT6, U1203 ISO6731FDWR, U1204 TPS70933DBVR, U1205 INA296A2IDR, U1206 SN74LVC1G08DBVR, U1301 DRV8353SRTAR, U1302 STM32G431CBT6, U1303 ISO6731FDWR, U1304 TPS70933DBVR, U1305 INA296A2IDR, U1306 SN74LVC1G08DBVR, U1401 DRV8353SRTAR, U1402 STM32G431CBT6, U1403 ISO6731FDWR, U1404 TPS70933DBVR, U1405 INA296A2IDR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

Commit message: Package ESC USB design for Quilter
Parts:
- removed C1130, C1230, C1330, C1430, C1530, C1630: 820u 100V, CP_Radial_D18.0mm_P7.50mm
- added C234: 1n 2kV, C_1206_3216Metric, F.Cu at (185.0, 7.97)
- added C235: 1n 2kV, C_1206_3216Metric, F.Cu at (185.0, 20.0)
- added J1104: USB_DFU_SERVICE, JST_GH_SM06B-GHS-TB_1x06-1MP_P1.25mm_Horizontal, F.Cu at (185.0, 32.0)
- added J1204: USB_DFU_SERVICE, JST_GH_SM06B-GHS-TB_1x06-1MP_P1.25mm_Horizontal, F.Cu at (185.0, 44.0)
- added J1304: USB_DFU_SERVICE, JST_GH_SM06B-GHS-TB_1x06-1MP_P1.25mm_Horizontal, F.Cu at (185.0, 56.0)
- added J1404: USB_DFU_SERVICE, JST_GH_SM06B-GHS-TB_1x06-1MP_P1.25mm_Horizontal, F.Cu at (185.0, 68.0)
- added J1504: USB_DFU_SERVICE, JST_GH_SM06B-GHS-TB_1x06-1MP_P1.25mm_Horizontal, F.Cu at (185.0, 80.0)
- added J1604: USB_DFU_SERVICE, JST_GH_SM06B-GHS-TB_1x06-1MP_P1.25mm_Horizontal, F.Cu at (185.0, 92.0)
- added J202: CTRL_USB_C, USB_C_Receptacle_GCT_USB4105-xx-A_16P_TopMnt_Horizontal, F.Cu at (185.0, 104.0)
- added J203: MOTOR_DFU_USB_C, USB_C_Receptacle_GCT_USB4105-xx-A_16P_TopMnt_Horizontal, F.Cu at (185.0, 116.0)
- added J204: SELECTED_CELL_BOOT_RESET, PinHeader_1x03_P2.54mm_Vertical, F.Cu at (185.0, 128.0)
- added R1180: 100k, R_0603_1608Metric, F.Cu at (185.0, 140.0)
- added R1181: 47k, R_0603_1608Metric, F.Cu at (217.0, 7.97)
- added R1182: 0, R_0603_1608Metric, F.Cu at (217.0, 20.0)
- added R1183: 0, R_0603_1608Metric, F.Cu at (217.0, 32.0)
- added R1184: 0, R_0603_1608Metric, F.Cu at (217.0, 44.0)
- added R1280: 100k, R_0603_1608Metric, F.Cu at (217.0, 56.0)
- added R1281: 47k, R_0603_1608Metric, F.Cu at (217.0, 68.0)
- added R1282: 0, R_0603_1608Metric, F.Cu at (217.0, 80.0)
- added R1283: 0, R_0603_1608Metric, F.Cu at (217.0, 92.0)
- added R1284: 0, R_0603_1608Metric, F.Cu at (217.0, 104.0)
- added R1380: 100k, R_0603_1608Metric, F.Cu at (217.0, 116.0)
- added R1381: 47k, R_0603_1608Metric, F.Cu at (217.0, 128.0)
- added R1382: 0, R_0603_1608Metric, F.Cu at (217.0, 140.0)
- added R1383: 0, R_0603_1608Metric, F.Cu at (249.0, 7.97)
- added R1384: 0, R_0603_1608Metric, F.Cu at (249.0, 20.0)
- added R1480: 100k, R_0603_1608Metric, F.Cu at (249.0, 32.0)
- added R1481: 47k, R_0603_1608Metric, F.Cu at (249.0, 44.0)
- added R1482: 0, R_0603_1608Metric, F.Cu at (249.0, 56.0)
- added R1483: 0, R_0603_1608Metric, F.Cu at (249.0, 68.0)
- added R1484: 0, R_0603_1608Metric, F.Cu at (249.0, 80.0)
- added R1580: 100k, R_0603_1608Metric, F.Cu at (249.0, 92.0)
- added R1581: 47k, R_0603_1608Metric, F.Cu at (249.0, 104.0)
- added R1582: 0, R_0603_1608Metric, F.Cu at (249.0, 116.0)
- added R1583: 0, R_0603_1608Metric, F.Cu at (249.0, 128.0)
- added R1584: 0, R_0603_1608Metric, F.Cu at (249.0, 140.0)
- added R1680: 100k, R_0603_1608Metric, F.Cu at (281.0, 7.97)
- added R1681: 47k, R_0603_1608Metric, F.Cu at (281.0, 20.0)
- added R1682: 0, R_0603_1608Metric, F.Cu at (281.0, 32.0)
- added R1683: 0, R_0603_1608Metric, F.Cu at (281.0, 44.0)
- added R1684: 0, R_0603_1608Metric, F.Cu at (281.0, 56.0)
- added R204: 5.1k, R_0603_1608Metric, F.Cu at (281.0, 68.0)
- added R205: 5.1k, R_0603_1608Metric, F.Cu at (281.0, 80.0)
- added R206: 27, R_0402_1005Metric, F.Cu at (281.0, 92.0)
- added R207: 27, R_0402_1005Metric, F.Cu at (281.0, 104.0)
- added R208: 100k, R_0603_1608Metric, F.Cu at (281.0, 116.0)
- added R209: 47k, R_0603_1608Metric, F.Cu at (281.0, 128.0)
- added R210: 1M, R_0603_1608Metric, F.Cu at (281.0, 140.0)
- added R211: 5.1k, R_0603_1608Metric, F.Cu at (313.0, 7.97)
- added R212: 5.1k, R_0603_1608Metric, F.Cu at (313.0, 20.0)
- added R213: 1M, R_0603_1608Metric, F.Cu at (313.0, 32.0)
- added SW201: 6P6T BBM SERVICE SELECTOR, PinHeader_2x21_P2.54mm_Vertical, F.Cu at (313.0, 44.0)
- added U1107: USBLC6-2SC6, SOT-23-6, F.Cu at (313.0, 56.0)
- added U1207: USBLC6-2SC6, SOT-23-6, F.Cu at (313.0, 68.0)
- added U1307: USBLC6-2SC6, SOT-23-6, F.Cu at (313.0, 80.0)
- added U1407: USBLC6-2SC6, SOT-23-6, F.Cu at (313.0, 92.0)
- added U1507: USBLC6-2SC6, SOT-23-6, F.Cu at (313.0, 104.0)
- added U1607: USBLC6-2SC6, SOT-23-6, F.Cu at (313.0, 116.0)
- added U208: USBLC6-2SC6, SOT-23-6, F.Cu at (313.0, 128.0)
- added U209: USBLC6-2SC6, SOT-23-6, F.Cu at (313.0, 140.0)
- moved R1455 741.7 mm to (4.06, 116.6), turned to 90 degrees
- moved R1155 739.7 mm to (4.06, 37.9), turned to 90 degrees
- moved R1453 731.6 mm to (4.05, 109.2), turned to -90 degrees
- moved C1133 730.3 mm to (16.2, 84.9), turned to 180 degrees
- moved R1109 726.2 mm to (11.0, 78.9), turned to 90 degrees
- moved R1406 716.1 mm to (5.08, 124.9), turned to 90 degrees
- moved R1410 710.8 mm to (36.1, 108.1), turned to 90 degrees
- moved R1106 709.7 mm to (10.1, 43.9)
- moved J1403 708.8 mm to (5.40, 96.2)
- moved R1110 708.7 mm to (36.1, 29.4), turned to 90 degrees
- moved Q1103 707.6 mm to (27.8, 29.0), turned to 90 degrees
- moved Q1403 707.3 mm to (27.8, 107.6), turned to 90 degrees
- moved R1409 707.2 mm to (30.5, 153.7)
- moved J1103 706.8 mm to (5.40, 17.6)
- moved R1445 704.5 mm to (12.7, 84.6), turned to 90 degrees
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Other:
- board size 150 x 150 mm -> 165 x 165 mm

Commit message: Keep ESC programming interface to two USB-C ports
Parts:
- removed J1104, J1204, J1304, J1404, J1504, J1604: USB_DFU_SERVICE, JST_GH_SM06B-GHS-TB_1x06-1MP_P1.25mm_Horizontal

Commit message: Replace ESC selector with seven-pin active-low control
Parts:
- removed J204: SELECTED_CELL_BOOT_RESET, PinHeader_1x03_P2.54mm_Vertical
- removed R1182, R1183, R1184, R1282, R1283, R1284, R1382, R1383, R1384, R1482, R1483, R1484, R1582, R1583, R1584, R1682, R1683, R1684: 0, R_0603_1608Metric
- added R214: 10k, R_0603_1608Metric, F.Cu at (185.0, 7.97)
- added R215: 10k, R_0603_1608Metric, F.Cu at (185.0, 20.0)
- added R216: 10k, R_0603_1608Metric, F.Cu at (185.0, 32.0)
- added R217: 10k, R_0603_1608Metric, F.Cu at (185.0, 44.0)
- added R218: 10k, R_0603_1608Metric, F.Cu at (185.0, 56.0)
- added R219: 10k, R_0603_1608Metric, F.Cu at (185.0, 68.0)
- SW201: value 6P6T BBM SERVICE SELECTOR -> 6-WAY ACTIVE-LOW SELECTOR; footprint PinHeader_2x21_P2.54mm_Vertical -> PinHeader_1x07_P2.54mm_Vertical
- moved J202 137.0 mm to (60.6, 161.3)
- moved SW201 129.8 mm to (243.6, 153.7)
- moved J203 65.3 mm to (138.1, 161.3)
- moved R1180 44.0 mm to (146.0, 160.2)
- moved C1501 15.0 mm to (77.5, 159.8)
- moved C1633 14.0 mm to (121.4, 161.9)
- moved C716 13.5 mm to (69.0, 160.2)
- moved C1660 13.1 mm to (128.8, 163.7)
- moved C1661 12.4 mm to (125.2, 162.0)
- moved C1422 12.2 mm to (47.8, 164.6)
- moved C1433 10.8 mm to (74.5, 162.5)
Connections:
- SW201 pad 1: /Controller and ADC/SVC_USB_DP -> /DGND
- SW201 pad 2: /Controller and ADC/SVC_USB_DM -> /Controller and ADC/SVC_CELL1_SEL_N
- SW201 pad 3: /Controller and ADC/SVC_USB_GND -> /Controller and ADC/SVC_CELL2_SEL_N
- SW201 pad 4: /Controller and ADC/SVC_USB_VBUS -> /Controller and ADC/SVC_CELL3_SEL_N
- SW201 pad 5: /Controller and ADC/SVC_USB_BOOT0 -> /Controller and ADC/SVC_CELL4_SEL_N
- SW201 pad 6: /Controller and ADC/SVC_USB_NRST -> /Controller and ADC/SVC_CELL5_SEL_N
- SW201 pad 7: /M1_USB_DP -> /Controller and ADC/SVC_CELL6_SEL_N
