File: hardware/esc/rev_b/controller.kicad_sch (KiCad schematic)
At the start: 47 parts, among them J201 ESC_SWD, U201 RP2354B, U204 TPS3430WDRCR, U205 SN74LVC1G08DBVR, U206 TCAN3413DR, U207 MCP2518FD-H/QBB, Y201 12MHz ABM8-272-T3, Y202 40MHz ABM8G

Commit message: Add ESC USB-C programming interfaces
Parts:
- added C234, C235: 1n 2kV, Capacitor_SMD:C_1206_3216Metric, symbol Device:C
- added J202: CTRL_USB_C, Connector_USB:USB_C_Receptacle_GCT_USB4105-xx-A_16P_TopMnt_Horizontal, symbol Connector:USB_C_Receptacle_USB2.0_16P
- added J203: MOTOR_DFU_USB_C, Connector_USB:USB_C_Receptacle_GCT_USB4105-xx-A_16P_TopMnt_Horizontal, symbol Connector:USB_C_Receptacle_USB2.0_16P
- added J204: SELECTED_CELL_BOOT_RESET, Connector_PinHeader_2.54mm:PinHeader_1x03_P2.54mm_Vertical, symbol Connector_Generic:Conn_01x03
- added R204, R205, R211, R212: 5.1k, Resistor_SMD:R_0603_1608Metric, symbol Device:R
- added R206, R207: 27, Resistor_SMD:R_0402_1005Metric, symbol Device:R
- added R208: 100k, Resistor_SMD:R_0603_1608Metric, symbol Device:R
- added R209: 47k, Resistor_SMD:R_0603_1608Metric, symbol Device:R
- added R210, R213: 1M, Resistor_SMD:R_0603_1608Metric, symbol Device:R
- added SW201: 6P6T BBM SERVICE SELECTOR, Connector_PinHeader_2.54mm:PinHeader_2x21_P2.54mm_Vertical, symbol revb:USB_CELL_SELECTOR_6P6T_BBM
- added U208, U209: USBLC6-2SC6, Package_TO_SOT_SMD:SOT-23-6, symbol revb:USBLC6-2SC6
- C201, C202, C203, C204, C205, C206, C207, C208, C209, C210, C211, C212, C213, C214, C215, C216, C217, C218, C219, C230, C231, C232, C233, C240, C241, C242, C243, D201, D202, FB201, FL201, J201, L201, R201, R202, R203, R231, R240, R241, R242, U201, U204, U205, U206, U207, Y201, Y202: hierarchy_path /98734485-5dd9-43e3-8e43-27cf828371fb/7fa4a6dc-f6d1-4938-a2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 -> /9645d861-d8e4-412a-9066-8076bbd6b1f6/377a6a3c-d3ed-4b65-82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
Connections:
- net DGND: now also C234.2, J202.A1 (GND), J202.A12 (GND), J202.B1 (GND), J202.B12 (GND), R204.2, R205.2, R209.2, R210.2, U208.2 (GND)
- net CTRL_USB_VBUS_SENSE: now reaches U201.20 (GPIO20)
- net CTRL_USB_VBUS_SENSE: now also R208.2, R209.1
- net CTRL_USB_DM_MCU: now reaches U201.66 (USB_DM)
- net CTRL_USB_DM_MCU: now also R206.2
- net CTRL_USB_DP_MCU: now reaches U201.67 (USB_DP)
- net CTRL_USB_DP_MCU: now also R207.2
- new net CTRL_USB_CC1: J202.A5 (CC1), R204.1
- new net CTRL_USB_CC2: J202.B5 (CC2), R205.1
- new net CTRL_USB_DM: R206.1, U208.6 (IO1)
- new net CTRL_USB_DM_CONN: J202.A7 (D-), J202.B7 (D-), U208.1 (IO1)
- new net CTRL_USB_DP: R207.1, U208.4 (IO2)
- new net CTRL_USB_DP_CONN: J202.A6 (D+), J202.B6 (D+), U208.3 (IO2)
- new net CTRL_USB_SHIELD: C234.1, J202.S1 (SHIELD), R210.1
- new net CTRL_USB_VBUS: J202.A4 (VBUS), J202.A9 (VBUS), J202.B4 (VBUS), J202.B9 (VBUS), R208.1, U208.5 (VBUS)
- new net M1_USB_BOOT0: SW201.11 (P1_5)
- new net M1_USB_DM: SW201.8 (P1_2)
- new net M1_USB_DP: SW201.7 (P1_1)
- new net M1_USB_GND: SW201.9 (P1_3)
- new net M1_USB_NRST: SW201.12 (P1_6)
- new net M1_USB_VBUS: SW201.10 (P1_4)
- new net M2_USB_BOOT0: SW201.17 (P2_5)
- new net M2_USB_DM: SW201.14 (P2_2)
- new net M2_USB_DP: SW201.13 (P2_1)
- new net M2_USB_GND: SW201.15 (P2_3)
- new net M2_USB_NRST: SW201.18 (P2_6)
- new net M2_USB_VBUS: SW201.16 (P2_4)
- new net M3_USB_BOOT0: SW201.23 (P3_5)
- new net M3_USB_DM: SW201.20 (P3_2)
- new net M3_USB_DP: SW201.19 (P3_1)
- new net M3_USB_GND: SW201.21 (P3_3)
- new net M3_USB_NRST: SW201.24 (P3_6)
- new net M3_USB_VBUS: SW201.22 (P3_4)
- new net M4_USB_BOOT0: SW201.29 (P4_5)
- new net M4_USB_DM: SW201.26 (P4_2)
- new net M4_USB_DP: SW201.25 (P4_1)
- new net M4_USB_GND: SW201.27 (P4_3)
- new net M4_USB_NRST: SW201.30 (P4_6)
- new net M4_USB_VBUS: SW201.28 (P4_4)
- new net M5_USB_BOOT0: SW201.35 (P5_5)
- new net M5_USB_DM: SW201.32 (P5_2)
- new net M5_USB_DP: SW201.31 (P5_1)
- new net M5_USB_GND: SW201.33 (P5_3)
- new net M5_USB_NRST: SW201.36 (P5_6)
- new net M5_USB_VBUS: SW201.34 (P5_4)
- new net M6_USB_BOOT0: SW201.41 (P6_5)
- new net M6_USB_DM: SW201.38 (P6_2)
- new net M6_USB_DP: SW201.37 (P6_1)
- new net M6_USB_GND: SW201.39 (P6_3)
- new net M6_USB_NRST: SW201.42 (P6_6)
- new net M6_USB_VBUS: SW201.40 (P6_4)
- new net SVC_USB_BOOT0: J204.1 (Pin_1), SW201.5 (COMMON_5)
- new net SVC_USB_CC1: J203.A5 (CC1), R211.1
- new net SVC_USB_CC2: J203.B5 (CC2), R212.1
- new net SVC_USB_DM: SW201.2 (COMMON_2), U209.6 (IO1)
- new net SVC_USB_DM_CONN: J203.A7 (D-), J203.B7 (D-), U209.1 (IO1)
- new net SVC_USB_DP: SW201.1 (COMMON_1), U209.4 (IO2)
- new net SVC_USB_DP_CONN: J203.A6 (D+), J203.B6 (D+), U209.3 (IO2)
- new net SVC_USB_GND: C235.2, J203.A1 (GND), J203.A12 (GND), J203.B1 (GND), J203.B12 (GND), J204.3 (Pin_3), R211.2, R212.2, R213.2, SW201.3 (COMMON_3), U209.2 (GND)
- new net SVC_USB_NRST: J204.2 (Pin_2), SW201.6 (COMMON_6)
- new net SVC_USB_SHIELD: C235.1, J203.S1 (SHIELD), R213.1
- new net SVC_USB_VBUS: J203.A4 (VBUS), J203.A9 (VBUS), J203.B4 (VBUS), J203.B9 (VBUS), SW201.4 (COMMON_4), U209.5 (VBUS)
- no-connect marks 40 -> 41
Other:
- note added: "SW201 MUST BE 6P6T BREAK-BEFORE-MAKE. Disconnect USB before changing position. Selector and harness must be rated for full cell-to-cell common-mode voltage."

Commit message: Keep ESC programming interface to two USB-C ports
Parts:
- C201, C202, C203, C204, C205, C206, C207, C208, C209, C210, C211, C212, C213, C214, C215, C216, C217, C218, C219, C230, C231, C232, C233, C234, C235, C240, C241, C242, C243, D201, D202, FB201, FL201, J201, J202, J203, J204, L201, R201, R202, R203, R204, R205, R206, R207, R208, R209, R210, R211, R212, R213, R231, R240, R241, R242, SW201, U201, U204, U205, U206, U207, U208, U209, Y201, Y202: hierarchy_path /9645d861-d8e4-412a-9066-8076bbd6b1f6/377a6a3c-d3ed-4b65-82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 -> /0143c865-039c-40ef-911e-d47147caf1a0/f4f56cbd-fac8-43a1-aa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

Commit message: Replace ESC selector with seven-pin active-low control
Parts:
- removed J204: SELECTED_CELL_BOOT_RESET, Connector_PinHeader_2.54mm:PinHeader_1x03_P2.54mm_Vertical, symbol Connector_Generic:Conn_01x03
- removed SW201: 6P6T BBM SERVICE SELECTOR, Connector_PinHeader_2.54mm:PinHeader_2x21_P2.54mm_Vertical, symbol revb:USB_CELL_SELECTOR_6P6T_BBM
- added R214, R215, R216, R217, R218, R219: 10k, Resistor_SMD:R_0603_1608Metric, symbol Device:R
- added SW201: 6-WAY ACTIVE-LOW SELECTOR, Connector_PinHeader_2.54mm:PinHeader_1x07_P2.54mm_Vertical, symbol revb:USB_CELL_SELECTOR_6WAY_ACTIVE_LOW
- C201, C202, C203, C204, C205, C206, C207, C208, C209, C210, C211, C212, C213, C214, C215, C216, C217, C218, C219, C230, C231, C232, C233, C234, C235, C240, C241, C242, C243, D201, D202, FB201, FL201, J201, J202, J203, L201, R201, R202, R203, R204, R205, R206, R207, R208, R209, R210, R211, R212, R213, R231, R240, R241, R242, U201, U204, U205, U206, U207, U208, U209, Y201, Y202: hierarchy_path /0143c865-039c-40ef-911e-d47147caf1a0/f4f56cbd-fac8-43a1-aa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 -> /5e323666-3ad9-4dd7-b28a-403d3185198c/9e40c478-f178-4dbc-81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
Connections:
- net SVC_USB_DM is gone; now on net SVC_USB_DM_CONN: U209.6 (IO1)
- net SVC_USB_DP is gone; now on net SVC_USB_DP_CONN: U209.4 (IO2)
- net 3V3: now also R214.1, R215.1, R216.1, R217.1, R218.1, R219.1
- net DGND: now also SW201.1 (GND)
- new net SVC_CELL1_SEL_N: R214.2, SW201.2 (CELL1_SEL_N)
- new net SVC_CELL2_SEL_N: R215.2, SW201.3 (CELL2_SEL_N)
- new net SVC_CELL3_SEL_N: R216.2, SW201.4 (CELL3_SEL_N)
- new net SVC_CELL4_SEL_N: R217.2, SW201.5 (CELL4_SEL_N)
- new net SVC_CELL5_SEL_N: R218.2, SW201.6 (CELL5_SEL_N)
- new net SVC_CELL6_SEL_N: R219.2, SW201.7 (CELL6_SEL_N)
Other:
- note added: "SW201 has one DGND common and six active-low outputs with individual pull-ups. These are CONTROL SIGNALS ONLY: an external galvanically isolated USB switching module must switch D+/D-/selected ground/VBUS/BOOT0/NRST and enforce break-before-make."
- note removed: "SW201 MUST BE 6P6T BREAK-BEFORE-MAKE. Disconnect USB before changing position. Selector and harness must be rated for full cell-to-cell common-mode voltage."
