File: hardware/esc/rev_b/motor_1.kicad_sch (KiCad schematic)
At the start: 100 parts, among them J1101 FUSED_BATTERY_TAP, J1102 MOTOR_PHASES, J1103 LOCAL_SWD, J1104 USB_DFU_SERVICE, Q1101 IPTC014N10NM5, Q1102 IPTC014N10NM5, Q1103 IPTC014N10NM5, Q1104 IPTC014N10NM5, Q1105 IPTC014N10NM5, Q1106 IPTC014N10NM5, U1101 DRV8353SRTAR, U1102 STM32G431CBT6, U1103 ISO6731FDWR, U1104 TPS70933DBVR, U1105 INA296A2IDR, U1106 SN74LVC1G08DBVR, U1107 USBLC6-2SC6, Y1101 8MHz ABM8G

Commit message: Keep ESC programming interface to two USB-C ports
Parts:
- removed J1104: USB_DFU_SERVICE, Connector_JST:JST_GH_SM06B-GHS-TB_1x06-1MP_P1.25mm_Horizontal, symbol Connector_Generic:Conn_01x06
- C1101, C1102, C1103, C1104, C1105, C1106, C1107, C1120, C1121, C1122, C1123, C1131, C1132, C1133, C1134, C1135, C1136, C1150, C1160, C1161, C1162, C1163, C1164, C1165, C1166, C1167, C1168, C1169, C1170, C1171, C1172, C1173, C1174, C1175, C1176, C1177, D1101, D1102, FB1101, J1101, J1102, J1103, PS1101, Q1101, Q1102, Q1103, Q1104, Q1105, Q1106, R1101, R1102, R1103, R1104, R1105, R1106, R1107, R1108, R1109, R1110, R1111, R1112, R1120, R1121, R1122, R1123, R1130, R1131, R1132, R1133, R1140, R1141, R1142, R1143, R1144, R1145, R1150, R1151, R1152, R1153, R1154, R1155, R1156, R1157, R1158, R1159, R1180, R1181, R1182, R1183, R1184, TH1, U1101, U1102, U1103, U1104, U1105, U1106, U1107, Y1101: hierarchy_path /9645d861-d8e4-412a-9066-8076bbd6b1f6/6f4ffbb4-5135-4088-8b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 -> /0143c865-039c-40ef-911e-d47147caf1a0/702e8499-4667-4363-81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

Commit message: Replace ESC selector with seven-pin active-low control
Parts:
- removed R1182, R1183, R1184: 0, Resistor_SMD:R_0603_1608Metric, symbol Device:R
- C1101, C1102, C1103, C1104, C1105, C1106, C1107, C1120, C1121, C1122, C1123, C1131, C1132, C1133, C1134, C1135, C1136, C1150, C1160, C1161, C1162, C1163, C1164, C1165, C1166, C1167, C1168, C1169, C1170, C1171, C1172, C1173, C1174, C1175, C1176, C1177, D1101, D1102, FB1101, J1101, J1102, J1103, PS1101, Q1101, Q1102, Q1103, Q1104, Q1105, Q1106, R1101, R1102, R1103, R1104, R1105, R1106, R1107, R1108, R1109, R1110, R1111, R1112, R1120, R1121, R1122, R1123, R1130, R1131, R1132, R1133, R1140, R1141, R1142, R1143, R1144, R1145, R1150, R1151, R1152, R1153, R1154, R1155, R1156, R1157, R1158, R1159, R1180, R1181, TH1, U1101, U1102, U1103, U1104, U1105, U1106, U1107, Y1101: hierarchy_path /0143c865-039c-40ef-911e-d47147caf1a0/702e8499-4667-4363-81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 -> /5e323666-3ad9-4dd7-b28a-403d3185198c/82b02ebb-fa40-47cf-9b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
