File: hardware/esc/rev_b/motor_2.kicad_sch (KiCad schematic)
At the start: 100 parts, among them J1201 FUSED_BATTERY_TAP, J1202 MOTOR_PHASES, J1203 LOCAL_SWD, J1204 USB_DFU_SERVICE, Q1201 IPTC014N10NM5, Q1202 IPTC014N10NM5, Q1203 IPTC014N10NM5, Q1204 IPTC014N10NM5, Q1205 IPTC014N10NM5, Q1206 IPTC014N10NM5, U1201 DRV8353SRTAR, U1202 STM32G431CBT6, U1203 ISO6731FDWR, U1204 TPS70933DBVR, U1205 INA296A2IDR, U1206 SN74LVC1G08DBVR, U1207 USBLC6-2SC6, Y1201 8MHz ABM8G

Commit message: Keep ESC programming interface to two USB-C ports
Parts:
- removed J1204: USB_DFU_SERVICE, Connector_JST:JST_GH_SM06B-GHS-TB_1x06-1MP_P1.25mm_Horizontal, symbol Connector_Generic:Conn_01x06
- C1201, C1202, C1203, C1204, C1205, C1206, C1207, C1220, C1221, C1222, C1223, C1231, C1232, C1233, C1234, C1235, C1236, C1250, C1260, C1261, C1262, C1263, C1264, C1265, C1266, C1267, C1268, C1269, C1270, C1271, C1272, C1273, C1274, C1275, C1276, C1277, D1201, D1202, FB1201, J1201, J1202, J1203, PS1201, Q1201, Q1202, Q1203, Q1204, Q1205, Q1206, R1201, R1202, R1203, R1204, R1205, R1206, R1207, R1208, R1209, R1210, R1211, R1212, R1220, R1221, R1222, R1223, R1230, R1231, R1232, R1233, R1240, R1241, R1242, R1243, R1244, R1245, R1250, R1251, R1252, R1253, R1254, R1255, R1256, R1257, R1258, R1259, R1280, R1281, R1282, R1283, R1284, TH2, U1201, U1202, U1203, U1204, U1205, U1206, U1207, Y1201: hierarchy_path /9645d861-d8e4-412a-9066-8076bbd6b1f6/d850c5a2-6df1-4c7e-b7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 -> /0143c865-039c-40ef-911e-d47147caf1a0/6b3a0005-60ca-42fb-94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

Commit message: Replace ESC selector with seven-pin active-low control
Parts:
- removed R1282, R1283, R1284: 0, Resistor_SMD:R_0603_1608Metric, symbol Device:R
- C1201, C1202, C1203, C1204, C1205, C1206, C1207, C1220, C1221, C1222, C1223, C1231, C1232, C1233, C1234, C1235, C1236, C1250, C1260, C1261, C1262, C1263, C1264, C1265, C1266, C1267, C1268, C1269, C1270, C1271, C1272, C1273, C1274, C1275, C1276, C1277, D1201, D1202, FB1201, J1201, J1202, J1203, PS1201, Q1201, Q1202, Q1203, Q1204, Q1205, Q1206, R1201, R1202, R1203, R1204, R1205, R1206, R1207, R1208, R1209, R1210, R1211, R1212, R1220, R1221, R1222, R1223, R1230, R1231, R1232, R1233, R1240, R1241, R1242, R1243, R1244, R1245, R1250, R1251, R1252, R1253, R1254, R1255, R1256, R1257, R1258, R1259, R1280, R1281, TH2, U1201, U1202, U1203, U1204, U1205, U1206, U1207, Y1201: hierarchy_path /0143c865-039c-40ef-911e-d47147caf1a0/6b3a0005-60ca-42fb-94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 -> /5e323666-3ad9-4dd7-b28a-403d3185198c/dcdcf72e-f1cb-4fcf-b6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
