File: hardware/esc/rev_b/motor_3.kicad_sch (KiCad schematic)
At the start: 100 parts, among them J1301 FUSED_BATTERY_TAP, J1302 MOTOR_PHASES, J1303 LOCAL_SWD, J1304 USB_DFU_SERVICE, Q1301 IPTC014N10NM5, Q1302 IPTC014N10NM5, Q1303 IPTC014N10NM5, Q1304 IPTC014N10NM5, Q1305 IPTC014N10NM5, Q1306 IPTC014N10NM5, U1301 DRV8353SRTAR, U1302 STM32G431CBT6, U1303 ISO6731FDWR, U1304 TPS70933DBVR, U1305 INA296A2IDR, U1306 SN74LVC1G08DBVR, U1307 USBLC6-2SC6, Y1301 8MHz ABM8G

Commit message: Keep ESC programming interface to two USB-C ports
Parts:
- removed J1304: USB_DFU_SERVICE, Connector_JST:JST_GH_SM06B-GHS-TB_1x06-1MP_P1.25mm_Horizontal, symbol Connector_Generic:Conn_01x06
- C1301, C1302, C1303, C1304, C1305, C1306, C1307, C1320, C1321, C1322, C1323, C1331, C1332, C1333, C1334, C1335, C1336, C1350, C1360, C1361, C1362, C1363, C1364, C1365, C1366, C1367, C1368, C1369, C1370, C1371, C1372, C1373, C1374, C1375, C1376, C1377, D1301, D1302, FB1301, J1301, J1302, J1303, PS1301, Q1301, Q1302, Q1303, Q1304, Q1305, Q1306, R1301, R1302, R1303, R1304, R1305, R1306, R1307, R1308, R1309, R1310, R1311, R1312, R1320, R1321, R1322, R1323, R1330, R1331, R1332, R1333, R1340, R1341, R1342, R1343, R1344, R1345, R1350, R1351, R1352, R1353, R1354, R1355, R1356, R1357, R1358, R1359, R1380, R1381, R1382, R1383, R1384, TH3, U1301, U1302, U1303, U1304, U1305, U1306, U1307, Y1301: hierarchy_path /9645d861-d8e4-412a-9066-8076bbd6b1f6/2646df52-a79d-4dd5-9a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 -> /0143c865-039c-40ef-911e-d47147caf1a0/736c94b1-1e95-4da5-9c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

Commit message: Replace ESC selector with seven-pin active-low control
Parts:
- removed R1382, R1383, R1384: 0, Resistor_SMD:R_0603_1608Metric, symbol Device:R
- C1301, C1302, C1303, C1304, C1305, C1306, C1307, C1320, C1321, C1322, C1323, C1331, C1332, C1333, C1334, C1335, C1336, C1350, C1360, C1361, C1362, C1363, C1364, C1365, C1366, C1367, C1368, C1369, C1370, C1371, C1372, C1373, C1374, C1375, C1376, C1377, D1301, D1302, FB1301, J1301, J1302, J1303, PS1301, Q1301, Q1302, Q1303, Q1304, Q1305, Q1306, R1301, R1302, R1303, R1304, R1305, R1306, R1307, R1308, R1309, R1310, R1311, R1312, R1320, R1321, R1322, R1323, R1330, R1331, R1332, R1333, R1340, R1341, R1342, R1343, R1344, R1345, R1350, R1351, R1352, R1353, R1354, R1355, R1356, R1357, R1358, R1359, R1380, R1381, TH3, U1301, U1302, U1303, U1304, U1305, U1306, U1307, Y1301: hierarchy_path /0143c865-039c-40ef-911e-d47147caf1a0/736c94b1-1e95-4da5-9c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 -> /5e323666-3ad9-4dd7-b28a-403d3185198c/de188998-b89e-4b7f-bc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
