File: hardware/esc/rev_b/motor_4.kicad_sch (KiCad schematic)
At the start: 100 parts, among them J1401 FUSED_BATTERY_TAP, J1402 MOTOR_PHASES, J1403 LOCAL_SWD, J1404 USB_DFU_SERVICE, Q1401 IPTC014N10NM5, Q1402 IPTC014N10NM5, Q1403 IPTC014N10NM5, Q1404 IPTC014N10NM5, Q1405 IPTC014N10NM5, Q1406 IPTC014N10NM5, U1401 DRV8353SRTAR, U1402 STM32G431CBT6, U1403 ISO6731FDWR, U1404 TPS70933DBVR, U1405 INA296A2IDR, U1406 SN74LVC1G08DBVR, U1407 USBLC6-2SC6, Y1401 8MHz ABM8G

Commit message: Keep ESC programming interface to two USB-C ports
Parts:
- removed J1404: USB_DFU_SERVICE, Connector_JST:JST_GH_SM06B-GHS-TB_1x06-1MP_P1.25mm_Horizontal, symbol Connector_Generic:Conn_01x06
- C1401, C1402, C1403, C1404, C1405, C1406, C1407, C1420, C1421, C1422, C1423, C1431, C1432, C1433, C1434, C1435, C1436, C1450, C1460, C1461, C1462, C1463, C1464, C1465, C1466, C1467, C1468, C1469, C1470, C1471, C1472, C1473, C1474, C1475, C1476, C1477, D1401, D1402, FB1401, J1401, J1402, J1403, PS1401, Q1401, Q1402, Q1403, Q1404, Q1405, Q1406, R1401, R1402, R1403, R1404, R1405, R1406, R1407, R1408, R1409, R1410, R1411, R1412, R1420, R1421, R1422, R1423, R1430, R1431, R1432, R1433, R1440, R1441, R1442, R1443, R1444, R1445, R1450, R1451, R1452, R1453, R1454, R1455, R1456, R1457, R1458, R1459, R1480, R1481, R1482, R1483, R1484, TH4, U1401, U1402, U1403, U1404, U1405, U1406, U1407, Y1401: hierarchy_path /9645d861-d8e4-412a-9066-8076bbd6b1f6/468fe66e-d6f5-40b9-aa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 -> /0143c865-039c-40ef-911e-d47147caf1a0/f6a66df9-9849-40ed-b9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

Commit message: Replace ESC selector with seven-pin active-low control
Parts:
- removed R1482, R1483, R1484: 0, Resistor_SMD:R_0603_1608Metric, symbol Device:R
- C1401, C1402, C1403, C1404, C1405, C1406, C1407, C1420, C1421, C1422, C1423, C1431, C1432, C1433, C1434, C1435, C1436, C1450, C1460, C1461, C1462, C1463, C1464, C1465, C1466, C1467, C1468, C1469, C1470, C1471, C1472, C1473, C1474, C1475, C1476, C1477, D1401, D1402, FB1401, J1401, J1402, J1403, PS1401, Q1401, Q1402, Q1403, Q1404, Q1405, Q1406, R1401, R1402, R1403, R1404, R1405, R1406, R1407, R1408, R1409, R1410, R1411, R1412, R1420, R1421, R1422, R1423, R1430, R1431, R1432, R1433, R1440, R1441, R1442, R1443, R1444, R1445, R1450, R1451, R1452, R1453, R1454, R1455, R1456, R1457, R1458, R1459, R1480, R1481, TH4, U1401, U1402, U1403, U1404, U1405, U1406, U1407, Y1401: hierarchy_path /0143c865-039c-40ef-911e-d47147caf1a0/f6a66df9-9849-40ed-b9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 -> /5e323666-3ad9-4dd7-b28a-403d3185198c/3f9c3405-670a-42f6-96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
