File: hardware/esc/rev_b/motor_5.kicad_sch (KiCad schematic)
At the start: 100 parts, among them J1501 FUSED_BATTERY_TAP, J1502 MOTOR_PHASES, J1503 LOCAL_SWD, J1504 USB_DFU_SERVICE, Q1501 IPTC014N10NM5, Q1502 IPTC014N10NM5, Q1503 IPTC014N10NM5, Q1504 IPTC014N10NM5, Q1505 IPTC014N10NM5, Q1506 IPTC014N10NM5, U1501 DRV8353SRTAR, U1502 STM32G431CBT6, U1503 ISO6731FDWR, U1504 TPS70933DBVR, U1505 INA296A2IDR, U1506 SN74LVC1G08DBVR, U1507 USBLC6-2SC6, Y1501 8MHz ABM8G

Commit message: Keep ESC programming interface to two USB-C ports
Parts:
- removed J1504: USB_DFU_SERVICE, Connector_JST:JST_GH_SM06B-GHS-TB_1x06-1MP_P1.25mm_Horizontal, symbol Connector_Generic:Conn_01x06
- C1501, C1502, C1503, C1504, C1505, C1506, C1507, C1520, C1521, C1522, C1523, C1531, C1532, C1533, C1534, C1535, C1536, C1550, C1560, C1561, C1562, C1563, C1564, C1565, C1566, C1567, C1568, C1569, C1570, C1571, C1572, C1573, C1574, C1575, C1576, C1577, D1501, D1502, FB1501, J1501, J1502, J1503, PS1501, Q1501, Q1502, Q1503, Q1504, Q1505, Q1506, R1501, R1502, R1503, R1504, R1505, R1506, R1507, R1508, R1509, R1510, R1511, R1512, R1520, R1521, R1522, R1523, R1530, R1531, R1532, R1533, R1540, R1541, R1542, R1543, R1544, R1545, R1550, R1551, R1552, R1553, R1554, R1555, R1556, R1557, R1558, R1559, R1580, R1581, R1582, R1583, R1584, TH5, U1501, U1502, U1503, U1504, U1505, U1506, U1507, Y1501: hierarchy_path /9645d861-d8e4-412a-9066-8076bbd6b1f6/0a8863de-3628-49a5-bb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 -> /0143c865-039c-40ef-911e-d47147caf1a0/0220997d-c325-4831-bb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

Commit message: Replace ESC selector with seven-pin active-low control
Parts:
- removed R1582, R1583, R1584: 0, Resistor_SMD:R_0603_1608Metric, symbol Device:R
- C1501, C1502, C1503, C1504, C1505, C1506, C1507, C1520, C1521, C1522, C1523, C1531, C1532, C1533, C1534, C1535, C1536, C1550, C1560, C1561, C1562, C1563, C1564, C1565, C1566, C1567, C1568, C1569, C1570, C1571, C1572, C1573, C1574, C1575, C1576, C1577, D1501, D1502, FB1501, J1501, J1502, J1503, PS1501, Q1501, Q1502, Q1503, Q1504, Q1505, Q1506, R1501, R1502, R1503, R1504, R1505, R1506, R1507, R1508, R1509, R1510, R1511, R1512, R1520, R1521, R1522, R1523, R1530, R1531, R1532, R1533, R1540, R1541, R1542, R1543, R1544, R1545, R1550, R1551, R1552, R1553, R1554, R1555, R1556, R1557, R1558, R1559, R1580, R1581, TH5, U1501, U1502, U1503, U1504, U1505, U1506, U1507, Y1501: hierarchy_path /0143c865-039c-40ef-911e-d47147caf1a0/0220997d-c325-4831-bb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 -> /5e323666-3ad9-4dd7-b28a-403d3185198c/0b53785b-714d-47e0-89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
