File: hardware/esc/rev_b/motor_6.kicad_sch (KiCad schematic)
At the start: 100 parts, among them J1601 FUSED_BATTERY_TAP, J1602 MOTOR_PHASES, J1603 LOCAL_SWD, J1604 USB_DFU_SERVICE, Q1601 IPTC014N10NM5, Q1602 IPTC014N10NM5, Q1603 IPTC014N10NM5, Q1604 IPTC014N10NM5, Q1605 IPTC014N10NM5, Q1606 IPTC014N10NM5, U1601 DRV8353SRTAR, U1602 STM32G431CBT6, U1603 ISO6731FDWR, U1604 TPS70933DBVR, U1605 INA296A2IDR, U1606 SN74LVC1G08DBVR, U1607 USBLC6-2SC6, Y1601 8MHz ABM8G

Commit message: Keep ESC programming interface to two USB-C ports
Parts:
- removed J1604: USB_DFU_SERVICE, Connector_JST:JST_GH_SM06B-GHS-TB_1x06-1MP_P1.25mm_Horizontal, symbol Connector_Generic:Conn_01x06
- C1601, C1602, C1603, C1604, C1605, C1606, C1607, C1620, C1621, C1622, C1623, C1631, C1632, C1633, C1634, C1635, C1636, C1650, C1660, C1661, C1662, C1663, C1664, C1665, C1666, C1667, C1668, C1669, C1670, C1671, C1672, C1673, C1674, C1675, C1676, C1677, D1601, D1602, FB1601, J1601, J1602, J1603, PS1601, Q1601, Q1602, Q1603, Q1604, Q1605, Q1606, R1601, R1602, R1603, R1604, R1605, R1606, R1607, R1608, R1609, R1610, R1611, R1612, R1620, R1621, R1622, R1623, R1630, R1631, R1632, R1633, R1640, R1641, R1642, R1643, R1644, R1645, R1650, R1651, R1652, R1653, R1654, R1655, R1656, R1657, R1658, R1659, R1680, R1681, R1682, R1683, R1684, TH6, U1601, U1602, U1603, U1604, U1605, U1606, U1607, Y1601: hierarchy_path /9645d861-d8e4-412a-9066-8076bbd6b1f6/1d5f9359-dc7b-47d9-a6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 -> /0143c865-039c-40ef-911e-d47147caf1a0/26a29475-8fe2-4487-b9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

Commit message: Replace ESC selector with seven-pin active-low control
Parts:
- removed R1682, R1683, R1684: 0, Resistor_SMD:R_0603_1608Metric, symbol Device:R
- C1601, C1602, C1603, C1604, C1605, C1606, C1607, C1620, C1621, C1622, C1623, C1631, C1632, C1633, C1634, C1635, C1636, C1650, C1660, C1661, C1662, C1663, C1664, C1665, C1666, C1667, C1668, C1669, C1670, C1671, C1672, C1673, C1674, C1675, C1676, C1677, D1601, D1602, FB1601, J1601, J1602, J1603, PS1601, Q1601, Q1602, Q1603, Q1604, Q1605, Q1606, R1601, R1602, R1603, R1604, R1605, R1606, R1607, R1608, R1609, R1610, R1611, R1612, R1620, R1621, R1622, R1623, R1630, R1631, R1632, R1633, R1640, R1641, R1642, R1643, R1644, R1645, R1650, R1651, R1652, R1653, R1654, R1655, R1656, R1657, R1658, R1659, R1680, R1681, TH6, U1601, U1602, U1603, U1604, U1605, U1606, U1607, Y1601: hierarchy_path /0143c865-039c-40ef-911e-d47147caf1a0/26a29475-8fe2-4487-b9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 -> /5e323666-3ad9-4dd7-b28a-403d3185198c/096ae313-f3f2-4d1e-a9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
