File: hardware/esc/rev_b/esc_rev_b.kicad_pcb (KiCad board)
At the start: 4 copper layers, 196 x 296 mm, 646 parts, among them J1101 FUSED_BATTERY_TAP, J1102 MOTOR_PHASES, J1103 LOCAL_SWD, J1201 FUSED_BATTERY_TAP, J1202 MOTOR_PHASES, J1203 LOCAL_SWD, J1301 FUSED_BATTERY_TAP, J1302 MOTOR_PHASES, J1303 LOCAL_SWD, J1401 FUSED_BATTERY_TAP, J1402 MOTOR_PHASES, J1403 LOCAL_SWD, J1501 FUSED_BATTERY_TAP, J1502 MOTOR_PHASES, J1503 LOCAL_SWD, J1601 FUSED_BATTERY_TAP, J1602 MOTOR_PHASES, J1603 LOCAL_SWD, J201 ESC_SWD, J701 AUX_BATTERY, J702 FLIGHT_CAN_POWER, Q1101 IPTC014N10NM5, Q1102 IPTC014N10NM5, Q1103 IPTC014N10NM5, Q1104 IPTC014N10NM5, Q1105 IPTC014N10NM5, Q1106 IPTC014N10NM5, Q1201 IPTC014N10NM5, Q1202 IPTC014N10NM5, Q1203 IPTC014N10NM5, Q1204 IPTC014N10NM5, Q1205 IPTC014N10NM5, Q1206 IPTC014N10NM5, Q1301 IPTC014N10NM5, Q1302 IPTC014N10NM5, Q1303 IPTC014N10NM5, Q1304 IPTC014N10NM5, Q1305 IPTC014N10NM5, Q1306 IPTC014N10NM5, Q1401 IPTC014N10NM5, Q1402 IPTC014N10NM5, Q1403 IPTC014N10NM5, Q1404 IPTC014N10NM5, Q1405 IPTC014N10NM5, Q1406 IPTC014N10NM5, Q1501 IPTC014N10NM5, Q1502 IPTC014N10NM5, Q1503 IPTC014N10NM5, Q1504 IPTC014N10NM5, Q1505 IPTC014N10NM5, Q1506 IPTC014N10NM5, Q1601 IPTC014N10NM5, Q1602 IPTC014N10NM5, Q1603 IPTC014N10NM5, Q1604 IPTC014N10NM5, Q1605 IPTC014N10NM5, Q1606 IPTC014N10NM5, U1101 DRV8353SRTAR, U1102 STM32G431CBT6, U1103 ISO6731FDWR, U1104 TPS70933DBVR, U1105 INA296A2IDR, U1106 SN74LVC1G08DBVR, U1201 DRV8353SRTAR, U1202 STM32G431CBT6, U1203 ISO6731FDWR, U1204 TPS70933DBVR, U1205 INA296A2IDR, U1206 SN74LVC1G08DBVR, U1301 DRV8353SRTAR, U1302 STM32G431CBT6, U1303 ISO6731FDWR, U1304 TPS70933DBVR, U1305 INA296A2IDR, U1306 SN74LVC1G08DBVR, U1401 DRV8353SRTAR, U1402 STM32G431CBT6, U1403 ISO6731FDWR, U1404 TPS70933DBVR, U1405 INA296A2IDR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

Commit message: esc: route matched external CAN pair
Routing:
- net /CANL: track 3.13 -> 132.1 mm, vias 0 -> 2
- net /CANH: track 9.16 -> 131.6 mm, vias 2 -> 3
Changed lines of the file:
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@@
+	)
+	(segment
+		(start 71.145 5.5)
+		(end 71.145 3.25)
+		(width 0.2)
+		(layer "F.Cu")
+		(net 18)
 	)
 	(segment
@@
 		(net 18)
 	)
+	(via
+		(at 71.145 5.5)
+		(size 0.6)
+		(drill 0.3)
+		(layers "F.Cu" "B.Cu")
+		(net 18)
+	)
 	(segment
 		(start 183.495 20)
@@
 	)
 	(segment
+		(start 80 8.6)
+		(end 71.145 5.5)
+		(width 0.2)
+		(layer "In1.Cu")
+		(net 18)
+	)
+	(segment
+		(start 180 8.6)
+		(end 80 8.6)
+		(width 0.2)
+		(layer "In1.Cu")
+		(net 18)
+	)
+	(segment
+		(start 188.2 15.7)
+		(end 180 8.6)
+		(width 0.2)
+		(layer "In1.Cu")
+		(net 18)
+	)
+	(segment
+		(start 72.395 7)
+		(end 72.395 3.25)
+		(width 0.2)
+		(layer "F.Cu")
+		(net 19)
+	)
+	(segment
+		(start 189.4825 18.799999)
+		(end 191 20)
+		(width 0.2)
+		(layer "F.Cu")
+		(net 19)
+	)
+	(segment
 		(start 189.4825 18.799999)
 		(end 187.145 16.724999)
@@
 		(net 19)
 	)
+	(via
+		(at 72.395 7)
+		(size 0.6)
+		(drill 0.3)
+		(layers "F.Cu" "B.Cu")
+		(net 19)
+	)
+	(via
+		(at 191 20)
+		(size 0.6)
+		(drill 0.3)
+		(layers "F.Cu" "B.Cu")
+		(net 19)
+	)
+	(segment
+		(start 191 20)
+		(end 181.5 10.5)
+		(width 0.2)
+		(layer "In1.Cu")
+		(net 19)
+	)
+	(segment
+		(start 80 10.5)
+		(end 72.395 7)
+		(width 0.2)
+		(layer "In1.Cu")
+		(net 19)
+	)
+	(segment
+		(start 181.5 10.5)
+		(end 80 10.5)
+		(width 0.2)
+		(layer "In1.Cu")
+		(net 19)
+	)

Commit message: esc: route CAN controller MOSI
Routing:
- net /Controller and ADC/CAN_MOSI: track 0.00 -> 98.5 mm, vias 0 -> 2
- net /Controller and ADC/STATUS_LED: track 19.0 -> 38.7 mm, vias 0 -> 2
- net /Controller and ADC/CAN_MISO: track 56.8 -> 75.3 mm
- net /Controller and ADC/CAN_SCK: track 64.1 -> 76.5 mm
Changed lines of the file:
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@@
 	(segment
 		(start 131.25 18.875)
-		(end 131.25 15.375)
+		(end 130.5 18.875)
 		(width 0.2)
 		(layer "F.Cu")
@@
 	)
 	(segment
-		(start 131.25 15.375)
-		(end 133.375 15.375)
-		(width 0.2)
-		(layer "F.Cu")
-		(net 24)
-	)
-	(segment
 		(start 174.625 13.75)
 		(end 174.625 14)
@@
 	)
 	(segment
+		(start 130.5 18.875)
+		(end 130.5 20.5)
+		(width 0.2)
+		(layer "F.Cu")
+		(net 24)
+	)
+	(segment
 		(start 134.45 18.849999)
 		(end 133.549999 18.849999)
@@
 	)
 	(via
-		(at 133.375 15.375)
+		(at 130.5 20.5)
 		(size 0.6)
 		(drill 0.3)
@@
 	)
 	(segment
-		(start 133.375 15.375)
+		(start 125.5 13.5)
+		(end 141.25 13.5)
+		(width 0.2)
+		(layer "In1.Cu")
+		(net 24)
+	)
+	(segment
+		(start 130.5 20.5)
+		(end 125.5 20.5)
+		(width 0.2)
+		(layer "In1.Cu")
+		(net 24)
+	)
+	(segment
+		(start 125.5 20.5)
+		(end 125.5 13.5)
+		(width 0.2)
+		(layer "In1.Cu")
+		(net 24)
+	)
+	(segment
+		(start 141.25 13.5)
 		(end 141.25 15.375)
 		(width 0.2)
-		(layer "B.Cu")
-		(net 24)
+		(layer "In1.Cu")
+		(net 24)
+	)
+	(segment
+		(start 134.45 18.45)
+		(end 127 18.45)
+		(width 0.2)
+		(layer "F.Cu")
+		(net 25)
+	)
+	(segment
+		(start 127 18.45)
+		(end 127 16.5)
+		(width 0.2)
+		(layer "F.Cu")
+		(net 25)
+	)
+	(segment
+		(start 185.3 20.8)
+		(end 185.3 17.85)
+		(width 0.2)
+		(layer "F.Cu")
+		(net 25)
+	)
+	(segment
+		(start 185.3 17.85)
+		(end 173.2 17.85)
+		(width 0.2)
+		(layer "F.Cu")
+		(net 25)
+	)
+	(via
+		(at 185.3 20.8)
+		(size 0.6)
+		(drill 0.3)
+		(layers "F.Cu" "B.Cu")
+		(net 25)
+	)
+	(via
+		(at 127 16.5)
+		(size 0.6)
+		(drill 0.3)
+		(layers "F.Cu" "B.Cu")
+		(net 25)
+	)
+	(segment
+		(start 127 16.5)
+		(end 127 26.5)
+		(width 0.2)
+		(layer "B.Cu")
+		(net 25)
+	)
+	(segment
+		(start 185.3 26.5)
+		(end 185.3 20.8)
+		(width 0.2)
+		(layer "B.Cu")
+		(net 25)
+	)
+	(segment
+		(start 127 26.5)
+		(end 185.3 26.5)
+		(width 0.2)
+		(layer "B.Cu")
+		(net 25)
 	)
 	(segment
 		(start 134.45 18.05)
-		(end 132 18.05)
+		(end 130.5 18.05)
+		(width 0.2)
+		(layer "F.Cu")
+		(net 26)
+	)
+	(segment
+		(start 130.5 18.05)
+		(end 130.5 16.5)
 		(width 0.2)
 		(layer "F.Cu")
@@
 	)
 	(via
-		(at 132 18.05)
+		(at 130.5 16.5)
 		(size 0.6)
 		(drill 0.3)
@@
 	)
 	(segment
+		(start 130.5 16.5)
+		(end 136 16.5)
+		(width 0.2)
+		(layer "B.Cu")
+		(net 26)
+	)
+	(segment
+		(start 136 25.5)
+		(end 133.5 25.5)
+		(width 0.2)
+		(layer "B.Cu")
+		(net 26)
+	)
+	(segment
 		(start 175.8 20.3)
 		(end 174.2 18.5)
@@
 	)
 	(segment
+		(start 136 16.5)
+		(end 136 25.5)
+		(width 0.2)
+		(layer "B.Cu")
+		(net 26)
+	)
+	(segment
 		(start 178 22.5)
 		(end 175.8 20.3)
-		(width 0.2)
-		(layer "B.Cu")
-		(net 26)
-	)
-	(segment
-		(start 132 18.05)
-		(end 133.5 25.5)
 		(width 0.2)
 		(layer "B.Cu")
@@
 	(segment
 		(start 130.58 6.1)
-		(end 130.58 21.25)
-		(width 0.2)
-		(layer "F.Cu")
-		(net 32)
-	)
-	(segment
-		(start 130.58 21.25)
-		(end 134.45 21.249999)
-		(width 0.2)
-		(layer "F.Cu")
-		(net 32)
-	)
+		(end 130.58 7.2)
+		(width 0.2)
+		(layer "F.Cu")
+		(net 32)
+	)
+	(segment
+		(start 130.8 22.5)
+		(end 130.8 21.25)
+		(width 0.2)
+		(layer "F.Cu")
+		(net 32)
+	)
+	(segment
+		(start 130.8 21.25)
+		(end 134.45 21.25)
+		(width 0.2)
+		(layer "F.Cu")
+		(net 32)
+	)
+	(via
+		(at 130.58 7.2)
+		(size 0.6)
+		(drill 0.3)
+		(layers "F.Cu" "B.Cu")
+		(net 32)
+	)
+	(via
+		(at 130.8 22.5)
+		(size 0.6)
+		(drill 0.3)
+		(layers "F.Cu" "B.Cu")
+		(net 32)
+	)
+	(segment
+		(start 130.58 7.2)
+		(end 122 7.2)
+		(width 0.2)
+		(layer "In2.Cu")
+		(net 32)
+	)
+	(segment
+		(start 122 7.2)
+		(end 122 22.5)
+		(width 0.2)
+		(layer "In2.Cu")
+		(net 32)
+	)
+	(segment
+		(start 122 22.5)
+		(end 130.8 22.5)
+		(width 0.2)
+		(layer "In2.Cu")
+		(net 32)
+	)

Commit message: esc: connect local 1V1 core links
Routing:
- net /Controller and ADC/1V1: track 0.00 -> 4.04 mm
Changed lines of the file:
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@@
+	)
+	(segment
+		(start 141.6 11.8)
+		(end 142.1025 10.55)
+		(width 0.2)
+		(layer "F.Cu")
+		(net 20)
+	)
+	(segment
+		(start 146.065 21.68)
+		(end 147.59 22.155)
+		(width 0.2)
+		(layer "F.Cu")
+		(net 20)
+	)
+	(segment
+		(start 141.6 12.9)
+		(end 141.6 11.8)
+		(width 0.2)
+		(layer "F.Cu")
+		(net 20)
 	)
 	(segment

Commit message: esc: connect remaining local 1V1 decouplers
Routing:
- net /Controller and ADC/1V1: track 4.04 -> 14.5 mm
Changed lines of the file:
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@@
+	)
+	(segment
+		(start 145.25 17.65)
+		(end 145.25 15.13)
+		(width 0.2)
+		(layer "F.Cu")
+		(net 20)
 	)
 	(segment
@@
 	)
 	(segment
+		(start 131.935 16.2)
+		(end 131.934999 17)
+		(width 0.2)
+		(layer "F.Cu")
+		(net 20)
+	)
+	(segment
+		(start 133.55 16.2)
+		(end 131.935 16.2)
+		(width 0.2)
+		(layer "F.Cu")
+		(net 20)
+	)
+	(segment
 		(start 146.065 21.68)
 		(end 147.59 22.155)
 		(width 0.2)
 		(layer "F.Cu")
+		(net 20)
+	)
+	(segment
+		(start 134.45 17.649999)
+		(end 133.55 17.65)
+		(width 0.2)
+		(layer "F.Cu")
+		(net 20)
+	)
+	(segment
+		(start 133.55 17.65)
+		(end 133.55 16.2)
+		(width 0.2)
+		(layer "F.Cu")
+		(net 20)
+	)
+	(segment
+		(start 144.35 17.649999)
+		(end 145.25 17.65)
+		(width 0.2)
+		(layer "F.Cu")
+		(net 20)
+	)
+	(segment
+		(start 145.25 15.13)
+		(end 147.565 15.129999)
+		(width 0.2)
+		(layer "F.Cu")
